File: Data/Trabbi Schematic/think_s02_hv_power.kicad_sch (KiCad schematic)
At the start: 8 parts, among them K1 Start Inhibit Relay A, M1 Main Motor AC, SW1 Battery Lock Switch, SW2 Main Current Switch, U1 Contactor Box, U2 Motor Controller (TIM)

Commit message: Fix label text justification for KiCad 9
Add (justify left) to all label and global_label effects.
KiCad 9 requires explicit text justification — without it,
label text is mispositioned relative to the label shape.

Co-Authored-By: Claude Opus 4.6 <noreply@anthropic.com>
Changed lines of the file:
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@@
   )
   (label "+114V_FUSED" (at 60.960 44.450 0)
-    (effects (font (size 1.27 1.27)))
+    (effects (font (size 1.27 1.27)) (justify left))
   )
   (wire (pts (xy 39.370 120.650) (xy 39.370 139.700))
@@
   )
   (label "-114V" (at 49.530 139.700 0)
-    (effects (font (size 1.27 1.27)))
+    (effects (font (size 1.27 1.27)) (justify left))
   )
   (wire (pts (xy 173.990 82.550) (xy 250.190 82.550))
@@
   )
   (label "+114V_TO_MC" (at 184.150 82.550 0)
-    (effects (font (size 1.27 1.27)))
+    (effects (font (size 1.27 1.27)) (justify left))
   )
   (label "-114V_TO_MC" (at 184.150 93.980 0)
-    (effects (font (size 1.27 1.27)))
+    (effects (font (size 1.27 1.27)) (justify left))
   )
   (wire (pts (xy 308.610 83.820) (xy 321.310 83.820))
@@
   )
   (label "L1" (at 318.770 83.820 0)
-    (effects (font (size 1.27 1.27)))
+    (effects (font (size 1.27 1.27)) (justify left))
   )
   (wire (pts (xy 308.610 97.790) (xy 321.310 97.790))
@@
   )
   (label "L2" (at 318.770 97.790 0)
-    (effects (font (size 1.27 1.27)))
+    (effects (font (size 1.27 1.27)) (justify left))
   )
   (wire (pts (xy 308.610 110.490) (xy 321.310 110.490))
@@
   )
   (label "L3" (at 318.770 110.490 0)
-    (effects (font (size 1.27 1.27)))
+    (effects (font (size 1.27 1.27)) (justify left))
   )
   (wire (pts (xy 361.950 121.920) (xy 347.980 121.920))
@@
   )
   (global_label "CHASSIS_GND" (shape input) (at 347.980 121.920 180)
-    (effects (font (size 1.27 1.27)))
+    (effects (font (size 1.27 1.27)) (justify left))
     (property "Intersheetrefs" "${INTERSHEET_REFS}" (at 347.980 121.920 0)
       (effects (font (size 1.27 1.27)) hide)
@@
   )
   (global_label "GND" (shape input) (at 149.860 144.780 270)
-    (effects (font (size 1.27 1.27)))
+    (effects (font (size 1.27 1.27)) (justify left))
     (property "Intersheetrefs" "${INTERSHEET_REFS}" (at 149.860 144.780 0)
       (effects (font (size 1.27 1.27)) hide)
@@
   )
   (global_label "CB_RUN" (shape bidirectional) (at 162.560 53.340 90)
-    (effects (font (size 1.27 1.27)))
+    (effects (font (size 1.27 1.27)) (justify left))
     (property "Intersheetrefs" "${INTERSHEET_REFS}" (at 162.560 53.340 0)
       (effects (font (size 1.27 1.27)) hide)
@@
   )
   (global_label "BMS_CMD" (shape bidirectional) (at 156.210 53.340 90)
-    (effects (font (size 1.27 1.27)))
+    (effects (font (size 1.27 1.27)) (justify left))
     (property "Intersheetrefs" "${INTERSHEET_REFS}" (at 156.210 53.340 0)
       (effects (font (size 1.27 1.27)) hide)
@@
   )
   (global_label "CHG_START" (shape bidirectional) (at 149.860 53.340 90)
-    (effects (font (size 1.27 1.27)))
+    (effects (font (size 1.27 1.27)) (justify left))
     (property "Intersheetrefs" "${INTERSHEET_REFS}" (at 149.860 53.340 0)
       (effects (font (size 1.27 1.27)) hide)
@@
   )
   (global_label "PREHEAT" (shape bidirectional) (at 143.510 53.340 90)
-    (effects (font (size 1.27 1.27)))
+    (effects (font (size 1.27 1.27)) (justify left))
     (property "Intersheetrefs" "${INTERSHEET_REFS}" (at 143.510 53.340 0)
       (effects (font (size 1.27 1.27)) hide)
@@
   )
   (global_label "CHARGE" (shape bidirectional) (at 137.160 53.340 90)
-    (effects (font (size 1.27 1.27)))
+    (effects (font (size 1.27 1.27)) (justify left))
     (property "Intersheetrefs" "${INTERSHEET_REFS}" (at 137.160 53.340 0)
       (effects (font (size 1.27 1.27)) hide)
@@
   )
   (global_label "DRIVE" (shape bidirectional) (at 299.720 54.610 90)
-    (effects (font (size 1.27 1.27)))
+    (effects (font (size 1.27 1.27)) (justify left))
     (property "Intersheetrefs" "${INTERSHEET_REFS}" (at 299.720 54.610 0)
       (effects (font (size 1.27 1.27)) hide)
@@
   )
   (global_label "START" (shape bidirectional) (at 295.910 54.610 90)
-    (effects (font (size 1.27 1.27)))
+    (effects (font (size 1.27 1.27)) (justify left))
     (property "Intersheetrefs" "${INTERSHEET_REFS}" (at 295.910 54.610 0)
       (effects (font (size 1.27 1.27)) hide)
@@
   )
   (global_label "DRIVE_RDY" (shape bidirectional) (at 290.830 54.610 90)
-    (effects (font (size 1.27 1.27)))
+    (effects (font (size 1.27 1.27)) (justify left))
     (property "Intersheetrefs" "${INTERSHEET_REFS}" (at 290.830 54.610 0)
       (effects (font (size 1.27 1.27)) hide)
@@
   )
   (global_label "FAULT" (shape bidirectional) (at 285.750 54.610 90)
-    (effects (font (size 1.27 1.27)))
+    (effects (font (size 1.27 1.27)) (justify left))
     (property "Intersheetrefs" "${INTERSHEET_REFS}" (at 285.750 54.610 0)
       (effects (font (size 1.27 1.27)) hide)
@@
   )
   (global_label "POWER" (shape bidirectional) (at 281.940 54.610 90)
-    (effects (font (size 1.27 1.27)))
+    (effects (font (size 1.27 1.27)) (justify left))
     (property "Intersheetrefs" "${INTERSHEET_REFS}" (at 281.940 54.610 0)
       (effects (font (size 1.27 1.27)) hide)
@@
   )
   (global_label "RED_PWR" (shape bidirectional) (at 276.860 54.610 90)
-    (effects (font (size 1.27 1.27)))
+    (effects (font (size 1.27 1.27)) (justify left))
     (property "Intersheetrefs" "${INTERSHEET_REFS}" (at 276.860 54.610 0)
       (effects (font (size 1.27 1.27)) hide)
@@
   )
   (global_label "BRAKE_SW" (shape bidirectional) (at 273.050 54.610 90)
-    (effects (font (size 1.27 1.27)))
+    (effects (font (size 1.27 1.27)) (justify left))
     (property "Intersheetrefs" "${INTERSHEET_REFS}" (at 273.050 54.610 0)
       (effects (font (size 1.27 1.27)) hide)
@@
   )
   (global_label "REVERSE" (shape bidirectional) (at 267.970 54.610 90)
-    (effects (font (size 1.27 1.27)))
+    (effects (font (size 1.27 1.27)) (justify left))
     (property "Intersheetrefs" "${INTERSHEET_REFS}" (at 267.970 54.610 0)
       (effects (font (size 1.27 1.27)) hide)
@@
   )
   (global_label "GEAR_LOCK" (shape bidirectional) (at 262.890 54.610 90)
-    (effects (font (size 1.27 1.27)))
+    (effects (font (size 1.27 1.27)) (justify left))
     (property "Intersheetrefs" "${INTERSHEET_REFS}" (at 262.890 54.610 0)
       (effects (font (size 1.27 1.27)) hide)
@@
   )
   (global_label "RAD_FAN_CMD" (shape bidirectional) (at 259.080 54.610 90)
-    (effects (font (size 1.27 1.27)))
+    (effects (font (size 1.27 1.27)) (justify left))
     (property "Intersheetrefs" "${INTERSHEET_REFS}" (at 259.080 54.610 0)
       (effects (font (size 1.27 1.27)) hide)
@@
   )
   (global_label "K_LINE" (shape bidirectional) (at 288.290 166.370 270)
-    (effects (font (size 1.27 1.27)))
+    (effects (font (size 1.27 1.27)) (justify left))
     (property "Intersheetrefs" "${INTERSHEET_REFS}" (at 288.290 166.370 0)
       (effects (font (size 1.27 1.27)) hide)
@@
   )
   (global_label "L_LINE" (shape bidirectional) (at 270.510 166.370 270)
-    (effects (font (size 1.27 1.27)))
+    (effects (font (size 1.27 1.27)) (justify left))
     (property "Intersheetrefs" "${INTERSHEET_REFS}" (at 270.510 166.370 0)
       (effects (font (size 1.27 1.27)) hide)
@@
   )
   (global_label "+12V_FROM_CB" (shape output) (at 184.150 106.680 0)
-    (effects (font (size 1.27 1.27)))
+    (effects (font (size 1.27 1.27)) (justify left))
     (property "Intersheetrefs" "${INTERSHEET_REFS}" (at 184.150 106.680 0)
       (effects (font (size 1.27 1.27)) hide)
@@
   )
   (global_label "+114V" (shape output) (at 184.150 118.110 0)
-    (effects (font (size 1.27 1.27)))
+    (effects (font (size 1.27 1.27)) (justify left))
     (property "Intersheetrefs" "${INTERSHEET_REFS}" (at 184.150 118.110 0)
       (effects (font (size 1.27 1.27)) hide)
@@
   )
   (global_label "+12V_F28_DRIVE" (shape bidirectional) (at 149.860 240.030 180)
-    (effects (font (size 1.27 1.27)))
+    (effects (font (size 1.27 1.27)) (justify left))
     (property "Intersheetrefs" "${INTERSHEET_REFS}" (at 149.860 240.030 0)
       (effects (font (size 1.27 1.27)) hide)

Commit message: Relay symbol for flasher, label justify set to auto
- Flasher Relay (Think:FLASHER_RELAY) now has coil+switch graphics
  matching the standard relay symbol style
- All relays (SPST, SPDT, Flasher) use consistent coil+switch body
- Remove (justify left) from all label and global_label effects —
  KiCad 9 auto-determines text alignment based on label orientation

Co-Authored-By: Claude Opus 4.6 <noreply@anthropic.com>
Changed lines of the file:
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@@
   )
   (label "+114V_FUSED" (at 60.960 44.450 0)
-    (effects (font (size 1.27 1.27)) (justify left))
+    (effects (font (size 1.27 1.27)))
   )
   (wire (pts (xy 39.370 120.650) (xy 39.370 139.700))
@@
   )
   (label "-114V" (at 49.530 139.700 0)
-    (effects (font (size 1.27 1.27)) (justify left))
+    (effects (font (size 1.27 1.27)))
   )
   (wire (pts (xy 173.990 82.550) (xy 250.190 82.550))
@@
   )
   (label "+114V_TO_MC" (at 184.150 82.550 0)
-    (effects (font (size 1.27 1.27)) (justify left))
+    (effects (font (size 1.27 1.27)))
   )
   (label "-114V_TO_MC" (at 184.150 93.980 0)
-    (effects (font (size 1.27 1.27)) (justify left))
+    (effects (font (size 1.27 1.27)))
   )
   (wire (pts (xy 308.610 83.820) (xy 321.310 83.820))
@@
   )
   (label "L1" (at 318.770 83.820 0)
-    (effects (font (size 1.27 1.27)) (justify left))
+    (effects (font (size 1.27 1.27)))
   )
   (wire (pts (xy 308.610 97.790) (xy 321.310 97.790))
@@
   )
   (label "L2" (at 318.770 97.790 0)
-    (effects (font (size 1.27 1.27)) (justify left))
+    (effects (font (size 1.27 1.27)))
   )
   (wire (pts (xy 308.610 110.490) (xy 321.310 110.490))
@@
   )
   (label "L3" (at 318.770 110.490 0)
-    (effects (font (size 1.27 1.27)) (justify left))
+    (effects (font (size 1.27 1.27)))
   )
   (wire (pts (xy 361.950 121.920) (xy 347.980 121.920))
@@
   )
   (global_label "CHASSIS_GND" (shape input) (at 347.980 121.920 180)
-    (effects (font (size 1.27 1.27)) (justify left))
+    (effects (font (size 1.27 1.27)))
     (property "Intersheetrefs" "${INTERSHEET_REFS}" (at 347.980 121.920 0)
       (effects (font (size 1.27 1.27)) hide)
@@
   )
   (global_label "GND" (shape input) (at 149.860 144.780 270)
-    (effects (font (size 1.27 1.27)) (justify left))
+    (effects (font (size 1.27 1.27)))
     (property "Intersheetrefs" "${INTERSHEET_REFS}" (at 149.860 144.780 0)
       (effects (font (size 1.27 1.27)) hide)
@@
   )
   (global_label "CB_RUN" (shape bidirectional) (at 162.560 53.340 90)
-    (effects (font (size 1.27 1.27)) (justify left))
+    (effects (font (size 1.27 1.27)))
     (property "Intersheetrefs" "${INTERSHEET_REFS}" (at 162.560 53.340 0)
       (effects (font (size 1.27 1.27)) hide)
@@
   )
   (global_label "BMS_CMD" (shape bidirectional) (at 156.210 53.340 90)
-    (effects (font (size 1.27 1.27)) (justify left))
+    (effects (font (size 1.27 1.27)))
     (property "Intersheetrefs" "${INTERSHEET_REFS}" (at 156.210 53.340 0)
       (effects (font (size 1.27 1.27)) hide)
@@
   )
   (global_label "CHG_START" (shape bidirectional) (at 149.860 53.340 90)
-    (effects (font (size 1.27 1.27)) (justify left))
+    (effects (font (size 1.27 1.27)))
     (property "Intersheetrefs" "${INTERSHEET_REFS}" (at 149.860 53.340 0)
       (effects (font (size 1.27 1.27)) hide)
@@
   )
   (global_label "PREHEAT" (shape bidirectional) (at 143.510 53.340 90)
-    (effects (font (size 1.27 1.27)) (justify left))
+    (effects (font (size 1.27 1.27)))
     (property "Intersheetrefs" "${INTERSHEET_REFS}" (at 143.510 53.340 0)
       (effects (font (size 1.27 1.27)) hide)
@@
   )
   (global_label "CHARGE" (shape bidirectional) (at 137.160 53.340 90)
-    (effects (font (size 1.27 1.27)) (justify left))
+    (effects (font (size 1.27 1.27)))
     (property "Intersheetrefs" "${INTERSHEET_REFS}" (at 137.160 53.340 0)
       (effects (font (size 1.27 1.27)) hide)
@@
   )
   (global_label "DRIVE" (shape bidirectional) (at 299.720 54.610 90)
-    (effects (font (size 1.27 1.27)) (justify left))
+    (effects (font (size 1.27 1.27)))
     (property "Intersheetrefs" "${INTERSHEET_REFS}" (at 299.720 54.610 0)
       (effects (font (size 1.27 1.27)) hide)
@@
   )
   (global_label "START" (shape bidirectional) (at 295.910 54.610 90)
-    (effects (font (size 1.27 1.27)) (justify left))
+    (effects (font (size 1.27 1.27)))
     (property "Intersheetrefs" "${INTERSHEET_REFS}" (at 295.910 54.610 0)
       (effects (font (size 1.27 1.27)) hide)
@@
   )
   (global_label "DRIVE_RDY" (shape bidirectional) (at 290.830 54.610 90)
-    (effects (font (size 1.27 1.27)) (justify left))
+    (effects (font (size 1.27 1.27)))
     (property "Intersheetrefs" "${INTERSHEET_REFS}" (at 290.830 54.610 0)
       (effects (font (size 1.27 1.27)) hide)
@@
   )
   (global_label "FAULT" (shape bidirectional) (at 285.750 54.610 90)
-    (effects (font (size 1.27 1.27)) (justify left))
+    (effects (font (size 1.27 1.27)))
     (property "Intersheetrefs" "${INTERSHEET_REFS}" (at 285.750 54.610 0)
       (effects (font (size 1.27 1.27)) hide)
@@
   )
   (global_label "POWER" (shape bidirectional) (at 281.940 54.610 90)
-    (effects (font (size 1.27 1.27)) (justify left))
+    (effects (font (size 1.27 1.27)))
     (property "Intersheetrefs" "${INTERSHEET_REFS}" (at 281.940 54.610 0)
       (effects (font (size 1.27 1.27)) hide)
@@
   )
   (global_label "RED_PWR" (shape bidirectional) (at 276.860 54.610 90)
-    (effects (font (size 1.27 1.27)) (justify left))
+    (effects (font (size 1.27 1.27)))
     (property "Intersheetrefs" "${INTERSHEET_REFS}" (at 276.860 54.610 0)
       (effects (font (size 1.27 1.27)) hide)
@@
   )
   (global_label "BRAKE_SW" (shape bidirectional) (at 273.050 54.610 90)
-    (effects (font (size 1.27 1.27)) (justify left))
+    (effects (font (size 1.27 1.27)))
     (property "Intersheetrefs" "${INTERSHEET_REFS}" (at 273.050 54.610 0)
       (effects (font (size 1.27 1.27)) hide)
@@
   )
   (global_label "REVERSE" (shape bidirectional) (at 267.970 54.610 90)
-    (effects (font (size 1.27 1.27)) (justify left))
+    (effects (font (size 1.27 1.27)))
     (property "Intersheetrefs" "${INTERSHEET_REFS}" (at 267.970 54.610 0)
       (effects (font (size 1.27 1.27)) hide)
@@
   )
   (global_label "GEAR_LOCK" (shape bidirectional) (at 262.890 54.610 90)
-    (effects (font (size 1.27 1.27)) (justify left))
+    (effects (font (size 1.27 1.27)))
     (property "Intersheetrefs" "${INTERSHEET_REFS}" (at 262.890 54.610 0)
       (effects (font (size 1.27 1.27)) hide)
@@
   )
   (global_label "RAD_FAN_CMD" (shape bidirectional) (at 259.080 54.610 90)
-    (effects (font (size 1.27 1.27)) (justify left))
+    (effects (font (size 1.27 1.27)))
     (property "Intersheetrefs" "${INTERSHEET_REFS}" (at 259.080 54.610 0)
       (effects (font (size 1.27 1.27)) hide)
@@
   )
   (global_label "K_LINE" (shape bidirectional) (at 288.290 166.370 270)
-    (effects (font (size 1.27 1.27)) (justify left))
+    (effects (font (size 1.27 1.27)))
     (property "Intersheetrefs" "${INTERSHEET_REFS}" (at 288.290 166.370 0)
       (effects (font (size 1.27 1.27)) hide)
@@
   )
   (global_label "L_LINE" (shape bidirectional) (at 270.510 166.370 270)
-    (effects (font (size 1.27 1.27)) (justify left))
+    (effects (font (size 1.27 1.27)))
     (property "Intersheetrefs" "${INTERSHEET_REFS}" (at 270.510 166.370 0)
       (effects (font (size 1.27 1.27)) hide)
@@
   )
   (global_label "+12V_FROM_CB" (shape output) (at 184.150 106.680 0)
-    (effects (font (size 1.27 1.27)) (justify left))
+    (effects (font (size 1.27 1.27)))
     (property "Intersheetrefs" "${INTERSHEET_REFS}" (at 184.150 106.680 0)
       (effects (font (size 1.27 1.27)) hide)
@@
   )
   (global_label "+114V" (shape output) (at 184.150 118.110 0)
-    (effects (font (size 1.27 1.27)) (justify left))
+    (effects (font (size 1.27 1.27)))
     (property "Intersheetrefs" "${INTERSHEET_REFS}" (at 184.150 118.110 0)
       (effects (font (size 1.27 1.27)) hide)
@@
   )
   (global_label "+12V_F28_DRIVE" (shape bidirectional) (at 149.860 240.030 180)
-    (effects (font (size 1.27 1.27)) (justify left))
+    (effects (font (size 1.27 1.27)))
     (property "Intersheetrefs" "${INTERSHEET_REFS}" (at 149.860 240.030 0)
       (effects (font (size 1.27 1.27)) hide)
