File: Data/Trabbi Schematic/think_s03_motor_ctrl.kicad_sch (KiCad schematic)
At the start: 9 parts, among them K1 Start Inhibit Relay B, K2 Radiator Fan Relay (R11), K3 Gear Lock Relay R8, K4 Gear Lock Relay R9, K5 Gear Lock Relay R10, M1 Gear Lock Motor E20/E21, SW1 Brake Light Switch (C12), U1 Motor Controller E01 Signals, U2 BMS (E02)

Commit message: Relay symbol for flasher, label justify set to auto
- Flasher Relay (Think:FLASHER_RELAY) now has coil+switch graphics
  matching the standard relay symbol style
- All relays (SPST, SPDT, Flasher) use consistent coil+switch body
- Remove (justify left) from all label and global_label effects —
  KiCad 9 auto-determines text alignment based on label orientation

Co-Authored-By: Claude Opus 4.6 <noreply@anthropic.com>
Changed lines of the file:
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@@
   )
   (global_label "DRIVE" (shape bidirectional) (at 72.390 73.660 180)
-    (effects (font (size 1.27 1.27)) (justify left))
+    (effects (font (size 1.27 1.27)))
     (property "Intersheetrefs" "${INTERSHEET_REFS}" (at 72.390 73.660 0)
       (effects (font (size 1.27 1.27)) hide)
@@
   )
   (global_label "START" (shape bidirectional) (at 72.390 82.550 180)
-    (effects (font (size 1.27 1.27)) (justify left))
+    (effects (font (size 1.27 1.27)))
     (property "Intersheetrefs" "${INTERSHEET_REFS}" (at 72.390 82.550 0)
       (effects (font (size 1.27 1.27)) hide)
@@
   )
   (global_label "DRIVE_RDY" (shape bidirectional) (at 72.390 91.440 180)
-    (effects (font (size 1.27 1.27)) (justify left))
+    (effects (font (size 1.27 1.27)))
     (property "Intersheetrefs" "${INTERSHEET_REFS}" (at 72.390 91.440 0)
       (effects (font (size 1.27 1.27)) hide)
@@
   )
   (global_label "FAULT" (shape bidirectional) (at 72.390 100.330 180)
-    (effects (font (size 1.27 1.27)) (justify left))
+    (effects (font (size 1.27 1.27)))
     (property "Intersheetrefs" "${INTERSHEET_REFS}" (at 72.390 100.330 0)
       (effects (font (size 1.27 1.27)) hide)
@@
   )
   (global_label "RED_PWR" (shape bidirectional) (at 72.390 109.220 180)
-    (effects (font (size 1.27 1.27)) (justify left))
+    (effects (font (size 1.27 1.27)))
     (property "Intersheetrefs" "${INTERSHEET_REFS}" (at 72.390 109.220 0)
       (effects (font (size 1.27 1.27)) hide)
@@
   )
   (global_label "BRAKE_SW" (shape bidirectional) (at 72.390 118.110 180)
-    (effects (font (size 1.27 1.27)) (justify left))
+    (effects (font (size 1.27 1.27)))
     (property "Intersheetrefs" "${INTERSHEET_REFS}" (at 72.390 118.110 0)
       (effects (font (size 1.27 1.27)) hide)
@@
   )
   (global_label "REVERSE" (shape bidirectional) (at 72.390 127.000 180)
-    (effects (font (size 1.27 1.27)) (justify left))
+    (effects (font (size 1.27 1.27)))
     (property "Intersheetrefs" "${INTERSHEET_REFS}" (at 72.390 127.000 0)
       (effects (font (size 1.27 1.27)) hide)
@@
   )
   (global_label "GEAR_LOCK" (shape bidirectional) (at 166.370 73.660 0)
-    (effects (font (size 1.27 1.27)) (justify left))
+    (effects (font (size 1.27 1.27)))
     (property "Intersheetrefs" "${INTERSHEET_REFS}" (at 166.370 73.660 0)
       (effects (font (size 1.27 1.27)) hide)
@@
   )
   (global_label "RAD_FAN_CMD" (shape bidirectional) (at 166.370 82.550 0)
-    (effects (font (size 1.27 1.27)) (justify left))
+    (effects (font (size 1.27 1.27)))
     (property "Intersheetrefs" "${INTERSHEET_REFS}" (at 166.370 82.550 0)
       (effects (font (size 1.27 1.27)) hide)
@@
   )
   (global_label "K_LINE" (shape bidirectional) (at 166.370 91.440 0)
-    (effects (font (size 1.27 1.27)) (justify left))
+    (effects (font (size 1.27 1.27)))
     (property "Intersheetrefs" "${INTERSHEET_REFS}" (at 166.370 91.440 0)
       (effects (font (size 1.27 1.27)) hide)
@@
   )
   (global_label "L_LINE" (shape bidirectional) (at 166.370 100.330 0)
-    (effects (font (size 1.27 1.27)) (justify left))
+    (effects (font (size 1.27 1.27)))
     (property "Intersheetrefs" "${INTERSHEET_REFS}" (at 166.370 100.330 0)
       (effects (font (size 1.27 1.27)) hide)
@@
   )
   (global_label "+12V_BAT" (shape output) (at 166.370 109.220 0)
-    (effects (font (size 1.27 1.27)) (justify left))
+    (effects (font (size 1.27 1.27)))
     (property "Intersheetrefs" "${INTERSHEET_REFS}" (at 166.370 109.220 0)
       (effects (font (size 1.27 1.27)) hide)
@@
   )
   (global_label "GND" (shape input) (at 166.370 118.110 0)
-    (effects (font (size 1.27 1.27)) (justify left))
+    (effects (font (size 1.27 1.27)))
     (property "Intersheetrefs" "${INTERSHEET_REFS}" (at 166.370 118.110 0)
       (effects (font (size 1.27 1.27)) hide)
@@
   )
   (global_label "POWER" (shape bidirectional) (at 166.370 127.000 0)
-    (effects (font (size 1.27 1.27)) (justify left))
+    (effects (font (size 1.27 1.27)))
     (property "Intersheetrefs" "${INTERSHEET_REFS}" (at 166.370 127.000 0)
       (effects (font (size 1.27 1.27)) hide)
@@
   )
   (global_label "BMS_CMD" (shape bidirectional) (at 156.210 208.280 0)
-    (effects (font (size 1.27 1.27)) (justify left))
+    (effects (font (size 1.27 1.27)))
     (property "Intersheetrefs" "${INTERSHEET_REFS}" (at 156.210 208.280 0)
       (effects (font (size 1.27 1.27)) hide)
@@
   )
   (global_label "CHG_STATUS_OK" (shape bidirectional) (at 156.210 215.900 0)
-    (effects (font (size 1.27 1.27)) (justify left))
+    (effects (font (size 1.27 1.27)))
     (property "Intersheetrefs" "${INTERSHEET_REFS}" (at 156.210 215.900 0)
       (effects (font (size 1.27 1.27)) hide)
@@
   )
   (global_label "K_LINE" (shape bidirectional) (at 156.210 223.520 0)
-    (effects (font (size 1.27 1.27)) (justify left))
+    (effects (font (size 1.27 1.27)))
     (property "Intersheetrefs" "${INTERSHEET_REFS}" (at 156.210 223.520 0)
       (effects (font (size 1.27 1.27)) hide)
@@
   )
   (global_label "L_LINE" (shape bidirectional) (at 156.210 231.140 0)
-    (effects (font (size 1.27 1.27)) (justify left))
+    (effects (font (size 1.27 1.27)))
     (property "Intersheetrefs" "${INTERSHEET_REFS}" (at 156.210 231.140 0)
       (effects (font (size 1.27 1.27)) hide)
@@
   )
   (global_label "BRAKE_SW" (shape bidirectional) (at 252.730 110.490 180)
-    (effects (font (size 1.27 1.27)) (justify left))
+    (effects (font (size 1.27 1.27)))
     (property "Intersheetrefs" "${INTERSHEET_REFS}" (at 252.730 110.490 0)
       (effects (font (size 1.27 1.27)) hide)
@@
   )
   (global_label "BRAKE_LIGHT_FEED" (shape bidirectional) (at 306.070 110.490 0)
-    (effects (font (size 1.27 1.27)) (justify left))
+    (effects (font (size 1.27 1.27)))
     (property "Intersheetrefs" "${INTERSHEET_REFS}" (at 306.070 110.490 0)
       (effects (font (size 1.27 1.27)) hide)
@@
   )
   (global_label "RAD_FAN_CMD" (shape bidirectional) (at 278.130 147.320 0)
-    (effects (font (size 1.27 1.27)) (justify left))
+    (effects (font (size 1.27 1.27)))
     (property "Intersheetrefs" "${INTERSHEET_REFS}" (at 278.130 147.320 0)
       (effects (font (size 1.27 1.27)) hide)
