File: Data/Trabbi Schematic/think_s06_bms_charger.kicad_sch (KiCad schematic)
At the start: 13 parts, among them J1 230V AC Mains Connection, K1 230V Relay, K2 Charge Cooling Relay R4, M1 Radiator Fan A (E11A), M2 Radiator Fan B (E11B), M3 Coolant Pump (E16), SW1 Charge Current Switch, U1 Battery Monitoring System (E0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, U2 Charger (E03)

Commit message: Relay symbol for flasher, label justify set to auto
- Flasher Relay (Think:FLASHER_RELAY) now has coil+switch graphics
  matching the standard relay symbol style
- All relays (SPST, SPDT, Flasher) use consistent coil+switch body
- Remove (justify left) from all label and global_label effects —
  KiCad 9 auto-determines text alignment based on label orientation

Co-Authored-By: Claude Opus 4.6 <noreply@anthropic.com>
Changed lines of the file:
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@@
   )
   (global_label "+12V_F28_DRIVE" (shape bidirectional) (at 59.690 83.820 180)
-    (effects (font (size 1.27 1.27)) (justify left))
+    (effects (font (size 1.27 1.27)))
     (property "Intersheetrefs" "${INTERSHEET_REFS}" (at 59.690 83.820 0)
       (effects (font (size 1.27 1.27)) hide)
@@
   )
   (global_label "GND" (shape input) (at 59.690 95.250 180)
-    (effects (font (size 1.27 1.27)) (justify left))
+    (effects (font (size 1.27 1.27)))
     (property "Intersheetrefs" "${INTERSHEET_REFS}" (at 59.690 95.250 0)
       (effects (font (size 1.27 1.27)) hide)
@@
   )
   (global_label "DC_LO_PWR" (shape bidirectional) (at 59.690 105.410 180)
-    (effects (font (size 1.27 1.27)) (justify left))
+    (effects (font (size 1.27 1.27)))
     (property "Intersheetrefs" "${INTERSHEET_REFS}" (at 59.690 105.410 0)
       (effects (font (size 1.27 1.27)) hide)
@@
   )
   (global_label "CHG_START_IN" (shape bidirectional) (at 59.690 116.840 180)
-    (effects (font (size 1.27 1.27)) (justify left))
+    (effects (font (size 1.27 1.27)))
     (property "Intersheetrefs" "${INTERSHEET_REFS}" (at 59.690 116.840 0)
       (effects (font (size 1.27 1.27)) hide)
@@
   )
   (global_label "CHG_STATUS_OK" (shape bidirectional) (at 140.970 82.550 0)
-    (effects (font (size 1.27 1.27)) (justify left))
+    (effects (font (size 1.27 1.27)))
     (property "Intersheetrefs" "${INTERSHEET_REFS}" (at 140.970 82.550 0)
       (effects (font (size 1.27 1.27)) hide)
@@
   )
   (global_label "CHG_START_OUT" (shape bidirectional) (at 140.970 91.440 0)
-    (effects (font (size 1.27 1.27)) (justify left))
+    (effects (font (size 1.27 1.27)))
     (property "Intersheetrefs" "${INTERSHEET_REFS}" (at 140.970 91.440 0)
       (effects (font (size 1.27 1.27)) hide)
@@
   )
   (global_label "BMS_CMD" (shape bidirectional) (at 140.970 100.330 0)
-    (effects (font (size 1.27 1.27)) (justify left))
+    (effects (font (size 1.27 1.27)))
     (property "Intersheetrefs" "${INTERSHEET_REFS}" (at 140.970 100.330 0)
       (effects (font (size 1.27 1.27)) hide)
@@
   )
   (global_label "K_LINE" (shape bidirectional) (at 140.970 109.220 0)
-    (effects (font (size 1.27 1.27)) (justify left))
+    (effects (font (size 1.27 1.27)))
     (property "Intersheetrefs" "${INTERSHEET_REFS}" (at 140.970 109.220 0)
       (effects (font (size 1.27 1.27)) hide)
@@
   )
   (global_label "L_LINE" (shape bidirectional) (at 140.970 118.110 0)
-    (effects (font (size 1.27 1.27)) (justify left))
+    (effects (font (size 1.27 1.27)))
     (property "Intersheetrefs" "${INTERSHEET_REFS}" (at 140.970 118.110 0)
       (effects (font (size 1.27 1.27)) hide)
@@
   )
   (global_label "CURR_S_12V" (shape bidirectional) (at 111.760 57.150 90)
-    (effects (font (size 1.27 1.27)) (justify left))
+    (effects (font (size 1.27 1.27)))
     (property "Intersheetrefs" "${INTERSHEET_REFS}" (at 111.760 57.150 0)
       (effects (font (size 1.27 1.27)) hide)
@@
   )
   (global_label "CURR_S_GND" (shape bidirectional) (at 104.140 57.150 90)
-    (effects (font (size 1.27 1.27)) (justify left))
+    (effects (font (size 1.27 1.27)))
     (property "Intersheetrefs" "${INTERSHEET_REFS}" (at 104.140 57.150 0)
       (effects (font (size 1.27 1.27)) hide)
@@
   )
   (global_label "CURR_SENSE" (shape bidirectional) (at 96.520 57.150 90)
-    (effects (font (size 1.27 1.27)) (justify left))
+    (effects (font (size 1.27 1.27)))
     (property "Intersheetrefs" "${INTERSHEET_REFS}" (at 96.520 57.150 0)
       (effects (font (size 1.27 1.27)) hide)
@@
   )
   (global_label "BATT_COOLING" (shape bidirectional) (at 88.900 57.150 90)
-    (effects (font (size 1.27 1.27)) (justify left))
+    (effects (font (size 1.27 1.27)))
     (property "Intersheetrefs" "${INTERSHEET_REFS}" (at 88.900 57.150 0)
       (effects (font (size 1.27 1.27)) hide)
@@
   )
   (label "TEMP1" (at 111.760 142.240 0)
-    (effects (font (size 1.27 1.27)) (justify left))
+    (effects (font (size 1.27 1.27)))
   )
   (wire (pts (xy 111.760 142.240) (xy 111.760 170.180))
@@
   )
   (label "TEMP2" (at 104.140 142.240 0)
-    (effects (font (size 1.27 1.27)) (justify left))
+    (effects (font (size 1.27 1.27)))
   )
   (wire (pts (xy 104.140 142.240) (xy 104.140 170.180))
@@
   )
   (label "TEMP3" (at 96.520 142.240 0)
-    (effects (font (size 1.27 1.27)) (justify left))
+    (effects (font (size 1.27 1.27)))
   )
   (wire (pts (xy 96.520 142.240) (xy 96.520 170.180))
@@
   )
   (label "TEMP4" (at 88.900 142.240 0)
-    (effects (font (size 1.27 1.27)) (justify left))
+    (effects (font (size 1.27 1.27)))
   )
   (wire (pts (xy 88.900 142.240) (xy 88.900 170.180))
@@
   )
   (label "L1_AC" (at 267.970 90.170 0)
-    (effects (font (size 1.27 1.27)) (justify left))
+    (effects (font (size 1.27 1.27)))
   )
   (wire (pts (xy 280.670 100.330) (xy 267.970 100.330))
@@
   )
   (label "L2_AC" (at 267.970 100.330 0)
-    (effects (font (size 1.27 1.27)) (justify left))
+    (effects (font (size 1.27 1.27)))
   )
   (wire (pts (xy 280.670 110.490) (xy 267.970 110.490))
@@
   )
   (label "GND_AC" (at 267.970 110.490 0)
-    (effects (font (size 1.27 1.27)) (justify left))
+    (effects (font (size 1.27 1.27)))
   )
   (wire (pts (xy 318.770 93.980) (xy 334.010 93.980))
@@
   )
   (global_label "+114V_CHARGER" (shape bidirectional) (at 334.010 93.980 0)
-    (effects (font (size 1.27 1.27)) (justify left))
+    (effects (font (size 1.27 1.27)))
     (property "Intersheetrefs" "${INTERSHEET_REFS}" (at 334.010 93.980 0)
       (effects (font (size 1.27 1.27)) hide)
@@
   )
   (global_label "-114V_CHARGER" (shape bidirectional) (at 334.010 106.680 0)
-    (effects (font (size 1.27 1.27)) (justify left))
+    (effects (font (size 1.27 1.27)))
     (property "Intersheetrefs" "${INTERSHEET_REFS}" (at 334.010 106.680 0)
       (effects (font (size 1.27 1.27)) hide)
@@
   )
   (global_label "CHG_START" (shape bidirectional) (at 304.800 63.500 90)
-    (effects (font (size 1.27 1.27)) (justify left))
+    (effects (font (size 1.27 1.27)))
     (property "Intersheetrefs" "${INTERSHEET_REFS}" (at 304.800 63.500 0)
       (effects (font (size 1.27 1.27)) hide)
@@
   )
   (global_label "CHG_STATUS_OK" (shape bidirectional) (at 294.640 63.500 90)
-    (effects (font (size 1.27 1.27)) (justify left))
+    (effects (font (size 1.27 1.27)))
     (property "Intersheetrefs" "${INTERSHEET_REFS}" (at 294.640 63.500 0)
       (effects (font (size 1.27 1.27)) hide)
@@
   )
   (global_label "K_LINE" (shape bidirectional) (at 304.800 137.160 270)
-    (effects (font (size 1.27 1.27)) (justify left))
+    (effects (font (size 1.27 1.27)))
     (property "Intersheetrefs" "${INTERSHEET_REFS}" (at 304.800 137.160 0)
       (effects (font (size 1.27 1.27)) hide)
@@
   )
   (global_label "L_LINE" (shape bidirectional) (at 294.640 137.160 270)
-    (effects (font (size 1.27 1.27)) (justify left))
+    (effects (font (size 1.27 1.27)))
     (property "Intersheetrefs" "${INTERSHEET_REFS}" (at 294.640 137.160 0)
       (effects (font (size 1.27 1.27)) hide)
@@
   )
   (label "230V_L1" (at 327.660 196.850 0)
-    (effects (font (size 1.27 1.27)) (justify left))
+    (effects (font (size 1.27 1.27)))
   )
   (wire (pts (xy 36.830 237.490) (xy 22.860 237.490))
@@
   )
   (global_label "BATT_COOLING" (shape bidirectional) (at 22.860 237.490 180)
-    (effects (font (size 1.27 1.27)) (justify left))
+    (effects (font (size 1.27 1.27)))
     (property "Intersheetrefs" "${INTERSHEET_REFS}" (at 22.860 237.490 0)
       (effects (font (size 1.27 1.27)) hide)
@@
   )
   (global_label "+12V_F6_RADFAN" (shape bidirectional) (at 77.470 229.870 180)
-    (effects (font (size 1.27 1.27)) (justify left))
+    (effects (font (size 1.27 1.27)))
     (property "Intersheetrefs" "${INTERSHEET_REFS}" (at 77.470 229.870 0)
       (effects (font (size 1.27 1.27)) hide)
@@
   )
   (global_label "GND" (shape input) (at 119.380 229.870 0)
-    (effects (font (size 1.27 1.27)) (justify left))
+    (effects (font (size 1.27 1.27)))
     (property "Intersheetrefs" "${INTERSHEET_REFS}" (at 119.380 229.870 0)
       (effects (font (size 1.27 1.27)) hide)
@@
   )
   (global_label "+12V_F6_RADFAN" (shape bidirectional) (at 77.470 255.270 180)
-    (effects (font (size 1.27 1.27)) (justify left))
+    (effects (font (size 1.27 1.27)))
     (property "Intersheetrefs" "${INTERSHEET_REFS}" (at 77.470 255.270 0)
       (effects (font (size 1.27 1.27)) hide)
@@
   )
   (global_label "GND" (shape input) (at 119.380 255.270 0)
-    (effects (font (size 1.27 1.27)) (justify left))
+    (effects (font (size 1.27 1.27)))
     (property "Intersheetrefs" "${INTERSHEET_REFS}" (at 119.380 255.270 0)
       (effects (font (size 1.27 1.27)) hide)
@@
   )
   (global_label "+12V_F10_WPUMP_CHG" (shape bidirectional) (at 176.530 240.030 180)
-    (effects (font (size 1.27 1.27)) (justify left))
+    (effects (font (size 1.27 1.27)))
     (property "Intersheetrefs" "${INTERSHEET_REFS}" (at 176.530 240.030 0)
       (effects (font (size 1.27 1.27)) hide)
@@
   )
   (global_label "GND" (shape input) (at 218.440 240.030 0)
-    (effects (font (size 1.27 1.27)) (justify left))
+    (effects (font (size 1.27 1.27)))
     (property "Intersheetrefs" "${INTERSHEET_REFS}" (at 218.440 240.030 0)
       (effects (font (size 1.27 1.27)) hide)
