File: Data/Trabbi Schematic/think_s08_rear_lights.kicad_sch (KiCad schematic)
At the start: 11 parts, among them K1 Reverse Light Relay R7, SW1 Brake Light Switch (C12)

Commit message: Add cross-sheet reference annotations to global labels
- Track all global label positions per sheet during build
- After building all sheets, annotate each global label with
  "→S01,S03,..." text showing which other sheets share the net
- 60 cross-sheet nets identified and annotated
- Two-pass build: 1) build all sheets 2) add cross-refs + save
- Text placed near label in 0.8mm font, offset to avoid overlap

Co-Authored-By: Claude Opus 4.6 <noreply@anthropic.com>
Other:
- note added: "→S01"
- note added: "→S01,S02,S03,S04,S05,S06,S07,S09,S10,S11,S12,S13"
- note added: "→S02,S03,S04,S11"
- note added: "→S03"
- note added: "→S09"
Changed lines of the file:
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@@
     (effects (font (size 1.000 1.000)))
+  )
+  (text "→S01" (at 50.340 59.650 0)
+    (effects (font (size 0.800 0.800)))
+  )
+  (text "→S02,S03,S04,S11" (at 50.340 64.730 0)
+    (effects (font (size 0.800 0.800)))
+  )
+  (text "→S01" (at 50.340 121.880 0)
+    (effects (font (size 0.800 0.800)))
+  )
+  (text "→S01" (at 50.340 132.040 0)
+    (effects (font (size 0.800 0.800)))
+  )
+  (text "→S01,S02,S03,S04,S05,S06,S07,S09,S10,S11,S12,S13" (at 246.840 41.870 0)
+    (effects (font (size 0.800 0.800)))
+  )
+  (text "→S01,S02,S03,S04,S05,S06,S07,S09,S10,S11,S12,S13" (at 246.840 62.190 0)
+    (effects (font (size 0.800 0.800)))
+  )
+  (text "→S01,S02,S03,S04,S05,S06,S07,S09,S10,S11,S12,S13" (at 246.840 102.830 0)
+    (effects (font (size 0.800 0.800)))
+  )
+  (text "→S01,S02,S03,S04,S05,S06,S07,S09,S10,S11,S12,S13" (at 246.840 121.880 0)
+    (effects (font (size 0.800 0.800)))
+  )
+  (text "→S01,S02,S03,S04,S05,S06,S07,S09,S10,S11,S12,S13" (at 249.380 147.280 0)
+    (effects (font (size 0.800 0.800)))
+  )
+  (text "→S01,S02,S03,S04,S05,S06,S07,S09,S10,S11,S12,S13" (at 246.840 177.760 0)
+    (effects (font (size 0.800 0.800)))
+  )
+  (text "→S01,S02,S03,S04,S05,S06,S07,S09,S10,S11,S12,S13" (at 246.840 198.080 0)
+    (effects (font (size 0.800 0.800)))
+  )
+  (text "→S01,S02,S03,S04,S05,S06,S07,S09,S10,S11,S12,S13" (at 246.840 227.290 0)
+    (effects (font (size 0.800 0.800)))
+  )
+  (text "→S01,S02,S03,S04,S05,S06,S07,S09,S10,S11,S12,S13" (at 373.840 121.880 0)
+    (effects (font (size 0.800 0.800)))
+  )
+  (text "→S09" (at 172.260 177.760 0)
+    (effects (font (size 0.800 0.800)))
+  )
+  (text "→S09" (at 172.260 198.080 0)
+    (effects (font (size 0.800 0.800)))
+  )
+  (text "→S01" (at 172.260 227.290 0)
+    (effects (font (size 0.800 0.800)))
+  )
+  (text "→S03" (at 327.200 121.880 0)
+    (effects (font (size 0.800 0.800)))
   )
   (symbol_instances)

Commit message: Fix label text justification for KiCad 9
Add (justify left) to all label and global_label effects.
KiCad 9 requires explicit text justification — without it,
label text is mispositioned relative to the label shape.

Co-Authored-By: Claude Opus 4.6 <noreply@anthropic.com>
Changed lines of the file:
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@@
   )
   (global_label "+12V_F15_HTDW_REV" (shape bidirectional) (at 53.340 57.150 180)
-    (effects (font (size 1.27 1.27)))
+    (effects (font (size 1.27 1.27)) (justify left))
     (property "Intersheetrefs" "${INTERSHEET_REFS}" (at 53.340 57.150 0)
       (effects (font (size 1.27 1.27)) hide)
@@
   )
   (global_label "REVERSE" (shape bidirectional) (at 53.340 62.230 180)
-    (effects (font (size 1.27 1.27)))
+    (effects (font (size 1.27 1.27)) (justify left))
     (property "Intersheetrefs" "${INTERSHEET_REFS}" (at 53.340 62.230 0)
       (effects (font (size 1.27 1.27)) hide)
@@
   )
   (global_label "+12V_F12_BRAKE" (shape bidirectional) (at 53.340 119.380 180)
-    (effects (font (size 1.27 1.27)))
+    (effects (font (size 1.27 1.27)) (justify left))
     (property "Intersheetrefs" "${INTERSHEET_REFS}" (at 53.340 119.380 0)
       (effects (font (size 1.27 1.27)) hide)
@@
   (junction (at 149.860 119.380) (diameter 0) (color 0 0 0 0))
   (global_label "+12V_F20_BRAKE2" (shape bidirectional) (at 53.340 129.540 180)
-    (effects (font (size 1.27 1.27)))
+    (effects (font (size 1.27 1.27)) (justify left))
     (property "Intersheetrefs" "${INTERSHEET_REFS}" (at 53.340 129.540 0)
       (effects (font (size 1.27 1.27)) hide)
@@
   )
   (global_label "GND" (shape input) (at 243.840 39.370 0)
-    (effects (font (size 1.27 1.27)))
+    (effects (font (size 1.27 1.27)) (justify left))
     (property "Intersheetrefs" "${INTERSHEET_REFS}" (at 243.840 39.370 0)
       (effects (font (size 1.27 1.27)) hide)
@@
   )
   (global_label "GND" (shape input) (at 243.840 59.690 0)
-    (effects (font (size 1.27 1.27)))
+    (effects (font (size 1.27 1.27)) (justify left))
     (property "Intersheetrefs" "${INTERSHEET_REFS}" (at 243.840 59.690 0)
       (effects (font (size 1.27 1.27)) hide)
@@
   )
   (global_label "GND" (shape input) (at 243.840 100.330 0)
-    (effects (font (size 1.27 1.27)))
+    (effects (font (size 1.27 1.27)) (justify left))
     (property "Intersheetrefs" "${INTERSHEET_REFS}" (at 243.840 100.330 0)
       (effects (font (size 1.27 1.27)) hide)
@@
   )
   (global_label "GND" (shape input) (at 243.840 119.380 0)
-    (effects (font (size 1.27 1.27)))
+    (effects (font (size 1.27 1.27)) (justify left))
     (property "Intersheetrefs" "${INTERSHEET_REFS}" (at 243.840 119.380 0)
       (effects (font (size 1.27 1.27)) hide)
@@
   )
   (global_label "GND" (shape input) (at 246.380 144.780 0)
-    (effects (font (size 1.27 1.27)))
+    (effects (font (size 1.27 1.27)) (justify left))
     (property "Intersheetrefs" "${INTERSHEET_REFS}" (at 246.380 144.780 0)
       (effects (font (size 1.27 1.27)) hide)
@@
   )
   (global_label "GND" (shape input) (at 243.840 175.260 0)
-    (effects (font (size 1.27 1.27)))
+    (effects (font (size 1.27 1.27)) (justify left))
     (property "Intersheetrefs" "${INTERSHEET_REFS}" (at 243.840 175.260 0)
       (effects (font (size 1.27 1.27)) hide)
@@
   )
   (global_label "GND" (shape input) (at 243.840 195.580 0)
-    (effects (font (size 1.27 1.27)))
+    (effects (font (size 1.27 1.27)) (justify left))
     (property "Intersheetrefs" "${INTERSHEET_REFS}" (at 243.840 195.580 0)
       (effects (font (size 1.27 1.27)) hide)
@@
   )
   (global_label "GND" (shape input) (at 243.840 224.790 0)
-    (effects (font (size 1.27 1.27)))
+    (effects (font (size 1.27 1.27)) (justify left))
     (property "Intersheetrefs" "${INTERSHEET_REFS}" (at 243.840 224.790 0)
       (effects (font (size 1.27 1.27)) hide)
@@
   )
   (global_label "TURN_SIG_LH_REAR" (shape bidirectional) (at 175.260 175.260 180)
-    (effects (font (size 1.27 1.27)))
+    (effects (font (size 1.27 1.27)) (justify left))
     (property "Intersheetrefs" "${INTERSHEET_REFS}" (at 175.260 175.260 0)
       (effects (font (size 1.27 1.27)) hide)
@@
   )
   (global_label "TURN_SIG_RH_REAR" (shape bidirectional) (at 175.260 195.580 180)
-    (effects (font (size 1.27 1.27)))
+    (effects (font (size 1.27 1.27)) (justify left))
     (property "Intersheetrefs" "${INTERSHEET_REFS}" (at 175.260 195.580 0)
       (effects (font (size 1.27 1.27)) hide)
@@
   )
   (global_label "+12V_F21_FOGR" (shape bidirectional) (at 175.260 224.790 180)
-    (effects (font (size 1.27 1.27)))
+    (effects (font (size 1.27 1.27)) (justify left))
     (property "Intersheetrefs" "${INTERSHEET_REFS}" (at 175.260 224.790 0)
       (effects (font (size 1.27 1.27)) hide)
@@
   )
   (global_label "BRAKE_LIGHT_FEED" (shape bidirectional) (at 330.200 119.380 180)
-    (effects (font (size 1.27 1.27)))
+    (effects (font (size 1.27 1.27)) (justify left))
     (property "Intersheetrefs" "${INTERSHEET_REFS}" (at 330.200 119.380 0)
       (effects (font (size 1.27 1.27)) hide)
@@
   )
   (global_label "GND" (shape input) (at 370.840 119.380 0)
-    (effects (font (size 1.27 1.27)))
+    (effects (font (size 1.27 1.27)) (justify left))
     (property "Intersheetrefs" "${INTERSHEET_REFS}" (at 370.840 119.380 0)
       (effects (font (size 1.27 1.27)) hide)

Commit message: Relay symbol for flasher, label justify set to auto
- Flasher Relay (Think:FLASHER_RELAY) now has coil+switch graphics
  matching the standard relay symbol style
- All relays (SPST, SPDT, Flasher) use consistent coil+switch body
- Remove (justify left) from all label and global_label effects —
  KiCad 9 auto-determines text alignment based on label orientation

Co-Authored-By: Claude Opus 4.6 <noreply@anthropic.com>
Changed lines of the file:
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@@
   )
   (global_label "+12V_F15_HTDW_REV" (shape bidirectional) (at 53.340 57.150 180)
-    (effects (font (size 1.27 1.27)) (justify left))
+    (effects (font (size 1.27 1.27)))
     (property "Intersheetrefs" "${INTERSHEET_REFS}" (at 53.340 57.150 0)
       (effects (font (size 1.27 1.27)) hide)
@@
   )
   (global_label "REVERSE" (shape bidirectional) (at 53.340 62.230 180)
-    (effects (font (size 1.27 1.27)) (justify left))
+    (effects (font (size 1.27 1.27)))
     (property "Intersheetrefs" "${INTERSHEET_REFS}" (at 53.340 62.230 0)
       (effects (font (size 1.27 1.27)) hide)
@@
   )
   (global_label "+12V_F12_BRAKE" (shape bidirectional) (at 53.340 119.380 180)
-    (effects (font (size 1.27 1.27)) (justify left))
+    (effects (font (size 1.27 1.27)))
     (property "Intersheetrefs" "${INTERSHEET_REFS}" (at 53.340 119.380 0)
       (effects (font (size 1.27 1.27)) hide)
@@
   (junction (at 149.860 119.380) (diameter 0) (color 0 0 0 0))
   (global_label "+12V_F20_BRAKE2" (shape bidirectional) (at 53.340 129.540 180)
-    (effects (font (size 1.27 1.27)) (justify left))
+    (effects (font (size 1.27 1.27)))
     (property "Intersheetrefs" "${INTERSHEET_REFS}" (at 53.340 129.540 0)
       (effects (font (size 1.27 1.27)) hide)
@@
   )
   (global_label "GND" (shape input) (at 243.840 39.370 0)
-    (effects (font (size 1.27 1.27)) (justify left))
+    (effects (font (size 1.27 1.27)))
     (property "Intersheetrefs" "${INTERSHEET_REFS}" (at 243.840 39.370 0)
       (effects (font (size 1.27 1.27)) hide)
@@
   )
   (global_label "GND" (shape input) (at 243.840 59.690 0)
-    (effects (font (size 1.27 1.27)) (justify left))
+    (effects (font (size 1.27 1.27)))
     (property "Intersheetrefs" "${INTERSHEET_REFS}" (at 243.840 59.690 0)
       (effects (font (size 1.27 1.27)) hide)
@@
   )
   (global_label "GND" (shape input) (at 243.840 100.330 0)
-    (effects (font (size 1.27 1.27)) (justify left))
+    (effects (font (size 1.27 1.27)))
     (property "Intersheetrefs" "${INTERSHEET_REFS}" (at 243.840 100.330 0)
       (effects (font (size 1.27 1.27)) hide)
@@
   )
   (global_label "GND" (shape input) (at 243.840 119.380 0)
-    (effects (font (size 1.27 1.27)) (justify left))
+    (effects (font (size 1.27 1.27)))
     (property "Intersheetrefs" "${INTERSHEET_REFS}" (at 243.840 119.380 0)
       (effects (font (size 1.27 1.27)) hide)
@@
   )
   (global_label "GND" (shape input) (at 246.380 144.780 0)
-    (effects (font (size 1.27 1.27)) (justify left))
+    (effects (font (size 1.27 1.27)))
     (property "Intersheetrefs" "${INTERSHEET_REFS}" (at 246.380 144.780 0)
       (effects (font (size 1.27 1.27)) hide)
@@
   )
   (global_label "GND" (shape input) (at 243.840 175.260 0)
-    (effects (font (size 1.27 1.27)) (justify left))
+    (effects (font (size 1.27 1.27)))
     (property "Intersheetrefs" "${INTERSHEET_REFS}" (at 243.840 175.260 0)
       (effects (font (size 1.27 1.27)) hide)
@@
   )
   (global_label "GND" (shape input) (at 243.840 195.580 0)
-    (effects (font (size 1.27 1.27)) (justify left))
+    (effects (font (size 1.27 1.27)))
     (property "Intersheetrefs" "${INTERSHEET_REFS}" (at 243.840 195.580 0)
       (effects (font (size 1.27 1.27)) hide)
@@
   )
   (global_label "GND" (shape input) (at 243.840 224.790 0)
-    (effects (font (size 1.27 1.27)) (justify left))
+    (effects (font (size 1.27 1.27)))
     (property "Intersheetrefs" "${INTERSHEET_REFS}" (at 243.840 224.790 0)
       (effects (font (size 1.27 1.27)) hide)
@@
   )
   (global_label "TURN_SIG_LH_REAR" (shape bidirectional) (at 175.260 175.260 180)
-    (effects (font (size 1.27 1.27)) (justify left))
+    (effects (font (size 1.27 1.27)))
     (property "Intersheetrefs" "${INTERSHEET_REFS}" (at 175.260 175.260 0)
       (effects (font (size 1.27 1.27)) hide)
@@
   )
   (global_label "TURN_SIG_RH_REAR" (shape bidirectional) (at 175.260 195.580 180)
-    (effects (font (size 1.27 1.27)) (justify left))
+    (effects (font (size 1.27 1.27)))
     (property "Intersheetrefs" "${INTERSHEET_REFS}" (at 175.260 195.580 0)
       (effects (font (size 1.27 1.27)) hide)
@@
   )
   (global_label "+12V_F21_FOGR" (shape bidirectional) (at 175.260 224.790 180)
-    (effects (font (size 1.27 1.27)) (justify left))
+    (effects (font (size 1.27 1.27)))
     (property "Intersheetrefs" "${INTERSHEET_REFS}" (at 175.260 224.790 0)
       (effects (font (size 1.27 1.27)) hide)
@@
   )
   (global_label "BRAKE_LIGHT_FEED" (shape bidirectional) (at 330.200 119.380 180)
-    (effects (font (size 1.27 1.27)) (justify left))
+    (effects (font (size 1.27 1.27)))
     (property "Intersheetrefs" "${INTERSHEET_REFS}" (at 330.200 119.380 0)
       (effects (font (size 1.27 1.27)) hide)
@@
   )
   (global_label "GND" (shape input) (at 370.840 119.380 0)
-    (effects (font (size 1.27 1.27)) (justify left))
+    (effects (font (size 1.27 1.27)))
     (property "Intersheetrefs" "${INTERSHEET_REFS}" (at 370.840 119.380 0)
       (effects (font (size 1.27 1.27)) hide)
