File: Data/Trabbi Schematic/think_s09_signals_horn.kicad_sch (KiCad schematic)
At the start: 15 parts, among them J1 Power Outlet (D60), K1 Flasher Relay R3, SW1 Horn Contact (steering wheel), SW2 Turn Signal / Hazard Switch (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, SW3 Driver Door Switch (C30), SW4 Passenger Door Switch (C31), SW5 Tailgate Switch (B10)

Commit message: Relay symbol for flasher, label justify set to auto
- Flasher Relay (Think:FLASHER_RELAY) now has coil+switch graphics
  matching the standard relay symbol style
- All relays (SPST, SPDT, Flasher) use consistent coil+switch body
- Remove (justify left) from all label and global_label effects —
  KiCad 9 auto-determines text alignment based on label orientation

Co-Authored-By: Claude Opus 4.6 <noreply@anthropic.com>
Changed lines of the file:
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@@
   )
   (global_label "+12V_F9_HORN_DOME" (shape bidirectional) (at 53.340 39.370 180)
-    (effects (font (size 1.27 1.27)) (justify left))
+    (effects (font (size 1.27 1.27)))
     (property "Intersheetrefs" "${INTERSHEET_REFS}" (at 53.340 39.370 0)
       (effects (font (size 1.27 1.27)) hide)
@@
   )
   (global_label "GND" (shape input) (at 106.680 39.370 0)
-    (effects (font (size 1.27 1.27)) (justify left))
+    (effects (font (size 1.27 1.27)))
     (property "Intersheetrefs" "${INTERSHEET_REFS}" (at 106.680 39.370 0)
       (effects (font (size 1.27 1.27)) hide)
@@
   )
   (global_label "+12V_F9_HORN_DOME" (shape bidirectional) (at 53.340 69.850 180)
-    (effects (font (size 1.27 1.27)) (justify left))
+    (effects (font (size 1.27 1.27)))
     (property "Intersheetrefs" "${INTERSHEET_REFS}" (at 53.340 69.850 0)
       (effects (font (size 1.27 1.27)) hide)
@@
   )
   (label "HORN_ACTIVE" (at 106.680 69.850 0)
-    (effects (font (size 1.27 1.27)) (justify left))
+    (effects (font (size 1.27 1.27)))
   )
   (wire (pts (xy 167.640 36.830) (xy 153.670 36.830))
@@
   )
   (global_label "+12V_F24_TURNSIG" (shape bidirectional) (at 153.670 36.830 180)
-    (effects (font (size 1.27 1.27)) (justify left))
+    (effects (font (size 1.27 1.27)))
     (property "Intersheetrefs" "${INTERSHEET_REFS}" (at 153.670 36.830 0)
       (effects (font (size 1.27 1.27)) hide)
@@
   )
   (global_label "GND" (shape input) (at 153.670 41.910 180)
-    (effects (font (size 1.27 1.27)) (justify left))
+    (effects (font (size 1.27 1.27)))
     (property "Intersheetrefs" "${INTERSHEET_REFS}" (at 153.670 41.910 0)
       (effects (font (size 1.27 1.27)) hide)
@@
   )
   (global_label "+12V_F24_TURNSIG" (shape bidirectional) (at 180.340 83.820 90)
-    (effects (font (size 1.27 1.27)) (justify left))
+    (effects (font (size 1.27 1.27)))
     (property "Intersheetrefs" "${INTERSHEET_REFS}" (at 180.340 83.820 0)
       (effects (font (size 1.27 1.27)) hide)
@@
   )
   (global_label "GND" (shape input) (at 323.850 80.010 0)
-    (effects (font (size 1.27 1.27)) (justify left))
+    (effects (font (size 1.27 1.27)))
     (property "Intersheetrefs" "${INTERSHEET_REFS}" (at 323.850 80.010 0)
       (effects (font (size 1.27 1.27)) hide)
@@
   )
   (global_label "GND" (shape input) (at 323.850 100.330 0)
-    (effects (font (size 1.27 1.27)) (justify left))
+    (effects (font (size 1.27 1.27)))
     (property "Intersheetrefs" "${INTERSHEET_REFS}" (at 323.850 100.330 0)
       (effects (font (size 1.27 1.27)) hide)
@@
   )
   (global_label "GND" (shape input) (at 323.850 124.460 0)
-    (effects (font (size 1.27 1.27)) (justify left))
+    (effects (font (size 1.27 1.27)))
     (property "Intersheetrefs" "${INTERSHEET_REFS}" (at 323.850 124.460 0)
       (effects (font (size 1.27 1.27)) hide)
@@
   )
   (global_label "GND" (shape input) (at 323.850 144.780 0)
-    (effects (font (size 1.27 1.27)) (justify left))
+    (effects (font (size 1.27 1.27)))
     (property "Intersheetrefs" "${INTERSHEET_REFS}" (at 323.850 144.780 0)
       (effects (font (size 1.27 1.27)) hide)
@@
   )
   (global_label "GND" (shape input) (at 323.850 170.180 0)
-    (effects (font (size 1.27 1.27)) (justify left))
+    (effects (font (size 1.27 1.27)))
     (property "Intersheetrefs" "${INTERSHEET_REFS}" (at 323.850 170.180 0)
       (effects (font (size 1.27 1.27)) hide)
@@
   )
   (global_label "GND" (shape input) (at 323.850 190.500 0)
-    (effects (font (size 1.27 1.27)) (justify left))
+    (effects (font (size 1.27 1.27)))
     (property "Intersheetrefs" "${INTERSHEET_REFS}" (at 323.850 190.500 0)
       (effects (font (size 1.27 1.27)) hide)
@@
   )
   (global_label "TURN_SIG_LH_REAR" (shape bidirectional) (at 274.320 170.180 180)
-    (effects (font (size 1.27 1.27)) (justify left))
+    (effects (font (size 1.27 1.27)))
     (property "Intersheetrefs" "${INTERSHEET_REFS}" (at 274.320 170.180 0)
       (effects (font (size 1.27 1.27)) hide)
@@
   )
   (global_label "TURN_SIG_RH_REAR" (shape bidirectional) (at 274.320 190.500 180)
-    (effects (font (size 1.27 1.27)) (justify left))
+    (effects (font (size 1.27 1.27)))
     (property "Intersheetrefs" "${INTERSHEET_REFS}" (at 274.320 190.500 0)
       (effects (font (size 1.27 1.27)) hide)
@@
   )
   (global_label "+12V_F9_HORN_DOME" (shape bidirectional) (at 52.070 170.180 180)
-    (effects (font (size 1.27 1.27)) (justify left))
+    (effects (font (size 1.27 1.27)))
     (property "Intersheetrefs" "${INTERSHEET_REFS}" (at 52.070 170.180 0)
       (effects (font (size 1.27 1.27)) hide)
@@
   )
   (label "DOME_SW" (at 107.950 170.180 0)
-    (effects (font (size 1.27 1.27)) (justify left))
+    (effects (font (size 1.27 1.27)))
   )
   (wire (pts (xy 69.850 199.390) (xy 53.340 199.390))
@@
   )
   (global_label "DOOR_SW_DRIVER" (shape bidirectional) (at 53.340 199.390 180)
-    (effects (font (size 1.27 1.27)) (justify left))
+    (effects (font (size 1.27 1.27)))
     (property "Intersheetrefs" "${INTERSHEET_REFS}" (at 53.340 199.390 0)
       (effects (font (size 1.27 1.27)) hide)
@@
   )
   (global_label "DOME_SW" (shape bidirectional) (at 106.680 199.390 0)
-    (effects (font (size 1.27 1.27)) (justify left))
+    (effects (font (size 1.27 1.27)))
     (property "Intersheetrefs" "${INTERSHEET_REFS}" (at 106.680 199.390 0)
       (effects (font (size 1.27 1.27)) hide)
@@
   )
   (global_label "DOOR_SW_PASS" (shape bidirectional) (at 53.340 219.710 180)
-    (effects (font (size 1.27 1.27)) (justify left))
+    (effects (font (size 1.27 1.27)))
     (property "Intersheetrefs" "${INTERSHEET_REFS}" (at 53.340 219.710 0)
       (effects (font (size 1.27 1.27)) hide)
@@
   )
   (global_label "DOME_SW" (shape bidirectional) (at 106.680 219.710 0)
-    (effects (font (size 1.27 1.27)) (justify left))
+    (effects (font (size 1.27 1.27)))
     (property "Intersheetrefs" "${INTERSHEET_REFS}" (at 106.680 219.710 0)
       (effects (font (size 1.27 1.27)) hide)
@@
   )
   (global_label "TAILGATE_SW" (shape bidirectional) (at 52.070 245.110 180)
-    (effects (font (size 1.27 1.27)) (justify left))
+    (effects (font (size 1.27 1.27)))
     (property "Intersheetrefs" "${INTERSHEET_REFS}" (at 52.070 245.110 0)
       (effects (font (size 1.27 1.27)) hide)
@@
   )
   (global_label "+12V_F8_OUTLET" (shape bidirectional) (at 271.780 229.870 180)
-    (effects (font (size 1.27 1.27)) (justify left))
+    (effects (font (size 1.27 1.27)))
     (property "Intersheetrefs" "${INTERSHEET_REFS}" (at 271.780 229.870 0)
       (effects (font (size 1.27 1.27)) hide)
@@
   )
   (global_label "GND" (shape input) (at 327.660 229.870 0)
-    (effects (font (size 1.27 1.27)) (justify left))
+    (effects (font (size 1.27 1.27)))
     (property "Intersheetrefs" "${INTERSHEET_REFS}" (at 327.660 229.870 0)
       (effects (font (size 1.27 1.27)) hide)
