File: Data/Trabbi Schematic/think_s10_wipers_alarm.kicad_sch (KiCad schematic)
At the start: 7 parts, among them K1 Wiper Relay R1, K2 Tailgate Release Relay R13, M1 Wiper Motor (E19), M2 Washer Pump (E10), SW1 Wiper Switch (C26), U1 Alarm Control Unit (P4)

Commit message: Relay symbol for flasher, label justify set to auto
- Flasher Relay (Think:FLASHER_RELAY) now has coil+switch graphics
  matching the standard relay symbol style
- All relays (SPST, SPDT, Flasher) use consistent coil+switch body
- Remove (justify left) from all label and global_label effects —
  KiCad 9 auto-determines text alignment based on label orientation

Co-Authored-By: Claude Opus 4.6 <noreply@anthropic.com>
Changed lines of the file:
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@@
   )
   (global_label "+12V_F14_WIPER" (shape bidirectional) (at 27.940 69.850 180)
-    (effects (font (size 1.27 1.27)) (justify left))
+    (effects (font (size 1.27 1.27)))
     (property "Intersheetrefs" "${INTERSHEET_REFS}" (at 27.940 69.850 0)
       (effects (font (size 1.27 1.27)) hide)
@@
   )
   (global_label "GND" (shape input) (at 287.020 63.500 0)
-    (effects (font (size 1.27 1.27)) (justify left))
+    (effects (font (size 1.27 1.27)))
     (property "Intersheetrefs" "${INTERSHEET_REFS}" (at 287.020 63.500 0)
       (effects (font (size 1.27 1.27)) hide)
@@
   )
   (label "WIPER_COM" (at 287.020 55.880 0)
-    (effects (font (size 1.27 1.27)) (justify left))
+    (effects (font (size 1.27 1.27)))
   )
   (wire (pts (xy 248.920 110.490) (xy 232.410 110.490))
@@
   )
   (global_label "+12V_F14_WIPER" (shape bidirectional) (at 232.410 110.490 180)
-    (effects (font (size 1.27 1.27)) (justify left))
+    (effects (font (size 1.27 1.27)))
     (property "Intersheetrefs" "${INTERSHEET_REFS}" (at 232.410 110.490 0)
       (effects (font (size 1.27 1.27)) hide)
@@
   )
   (global_label "GND" (shape input) (at 288.290 110.490 0)
-    (effects (font (size 1.27 1.27)) (justify left))
+    (effects (font (size 1.27 1.27)))
     (property "Intersheetrefs" "${INTERSHEET_REFS}" (at 288.290 110.490 0)
       (effects (font (size 1.27 1.27)) hide)
@@
   )
   (global_label "DOOR_DR" (shape bidirectional) (at 87.630 179.070 180)
-    (effects (font (size 1.27 1.27)) (justify left))
+    (effects (font (size 1.27 1.27)))
     (property "Intersheetrefs" "${INTERSHEET_REFS}" (at 87.630 179.070 0)
       (effects (font (size 1.27 1.27)) hide)
@@
   )
   (global_label "DOOR_PS" (shape bidirectional) (at 87.630 186.690 180)
-    (effects (font (size 1.27 1.27)) (justify left))
+    (effects (font (size 1.27 1.27)))
     (property "Intersheetrefs" "${INTERSHEET_REFS}" (at 87.630 186.690 0)
       (effects (font (size 1.27 1.27)) hide)
@@
   )
   (global_label "TAILGATE" (shape bidirectional) (at 87.630 194.310 180)
-    (effects (font (size 1.27 1.27)) (justify left))
+    (effects (font (size 1.27 1.27)))
     (property "Intersheetrefs" "${INTERSHEET_REFS}" (at 87.630 194.310 0)
       (effects (font (size 1.27 1.27)) hide)
@@
   )
   (global_label "+12V_F17_COLL_ALM" (shape bidirectional) (at 87.630 201.930 180)
-    (effects (font (size 1.27 1.27)) (justify left))
+    (effects (font (size 1.27 1.27)))
     (property "Intersheetrefs" "${INTERSHEET_REFS}" (at 87.630 201.930 0)
       (effects (font (size 1.27 1.27)) hide)
@@
   )
   (global_label "SIREN_OUT" (shape bidirectional) (at 151.130 177.800 0)
-    (effects (font (size 1.27 1.27)) (justify left))
+    (effects (font (size 1.27 1.27)))
     (property "Intersheetrefs" "${INTERSHEET_REFS}" (at 151.130 177.800 0)
       (effects (font (size 1.27 1.27)) hide)
@@
   )
   (global_label "TURN_SIG_ALARM" (shape bidirectional) (at 151.130 184.150 0)
-    (effects (font (size 1.27 1.27)) (justify left))
+    (effects (font (size 1.27 1.27)))
     (property "Intersheetrefs" "${INTERSHEET_REFS}" (at 151.130 184.150 0)
       (effects (font (size 1.27 1.27)) hide)
@@
   )
   (global_label "IGN_SENSE" (shape bidirectional) (at 151.130 190.500 0)
-    (effects (font (size 1.27 1.27)) (justify left))
+    (effects (font (size 1.27 1.27)))
     (property "Intersheetrefs" "${INTERSHEET_REFS}" (at 151.130 190.500 0)
       (effects (font (size 1.27 1.27)) hide)
@@
   )
   (global_label "DOOR_LOCK" (shape bidirectional) (at 151.130 196.850 0)
-    (effects (font (size 1.27 1.27)) (justify left))
+    (effects (font (size 1.27 1.27)))
     (property "Intersheetrefs" "${INTERSHEET_REFS}" (at 151.130 196.850 0)
       (effects (font (size 1.27 1.27)) hide)
@@
   )
   (global_label "DOOR_UNLOCK" (shape bidirectional) (at 151.130 203.200 0)
-    (effects (font (size 1.27 1.27)) (justify left))
+    (effects (font (size 1.27 1.27)))
     (property "Intersheetrefs" "${INTERSHEET_REFS}" (at 151.130 203.200 0)
       (effects (font (size 1.27 1.27)) hide)
@@
   )
   (global_label "GND" (shape input) (at 119.380 224.790 270)
-    (effects (font (size 1.27 1.27)) (justify left))
+    (effects (font (size 1.27 1.27)))
     (property "Intersheetrefs" "${INTERSHEET_REFS}" (at 119.380 224.790 0)
       (effects (font (size 1.27 1.27)) hide)
@@
   )
   (global_label "SIREN_OUT" (shape bidirectional) (at 236.220 209.550 180)
-    (effects (font (size 1.27 1.27)) (justify left))
+    (effects (font (size 1.27 1.27)))
     (property "Intersheetrefs" "${INTERSHEET_REFS}" (at 236.220 209.550 0)
       (effects (font (size 1.27 1.27)) hide)
@@
   )
   (global_label "GND" (shape input) (at 284.480 209.550 0)
-    (effects (font (size 1.27 1.27)) (justify left))
+    (effects (font (size 1.27 1.27)))
     (property "Intersheetrefs" "${INTERSHEET_REFS}" (at 284.480 209.550 0)
       (effects (font (size 1.27 1.27)) hide)
@@
   )
   (global_label "+12V_F9_HORN_DOME" (shape bidirectional) (at 233.680 167.640 180)
-    (effects (font (size 1.27 1.27)) (justify left))
+    (effects (font (size 1.27 1.27)))
     (property "Intersheetrefs" "${INTERSHEET_REFS}" (at 233.680 167.640 0)
       (effects (font (size 1.27 1.27)) hide)
@@
   )
   (global_label "TAILGATE_RELEASE" (shape bidirectional) (at 287.020 167.640 0)
-    (effects (font (size 1.27 1.27)) (justify left))
+    (effects (font (size 1.27 1.27)))
     (property "Intersheetrefs" "${INTERSHEET_REFS}" (at 287.020 167.640 0)
       (effects (font (size 1.27 1.27)) hide)
@@
   )
   (global_label "DOOR_SW_DRIVER" (shape bidirectional) (at 87.630 171.450 180)
-    (effects (font (size 1.27 1.27)) (justify left))
+    (effects (font (size 1.27 1.27)))
     (property "Intersheetrefs" "${INTERSHEET_REFS}" (at 87.630 171.450 0)
       (effects (font (size 1.27 1.27)) hide)
@@
   )
   (global_label "DOOR_SW_PASS" (shape bidirectional) (at 87.630 179.070 180)
-    (effects (font (size 1.27 1.27)) (justify left))
+    (effects (font (size 1.27 1.27)))
     (property "Intersheetrefs" "${INTERSHEET_REFS}" (at 87.630 179.070 0)
       (effects (font (size 1.27 1.27)) hide)
@@
   )
   (global_label "TAILGATE_SW" (shape bidirectional) (at 87.630 186.690 180)
-    (effects (font (size 1.27 1.27)) (justify left))
+    (effects (font (size 1.27 1.27)))
     (property "Intersheetrefs" "${INTERSHEET_REFS}" (at 87.630 186.690 0)
       (effects (font (size 1.27 1.27)) hide)
