File: Data/Trabbi Schematic/think_s11_diag_speed.kicad_sch (KiCad schematic)
At the start: 5 parts, among them J1 Diagnostic Connector (C09), J2 Multi-connector D01/D02/D03, K1 Charge Cooling Relay R4, U1 Collision Sensor (C050), U2 Speed Signal

Commit message: Add cross-sheet reference annotations to global labels
- Track all global label positions per sheet during build
- After building all sheets, annotate each global label with
  "→S01,S03,..." text showing which other sheets share the net
- 60 cross-sheet nets identified and annotated
- Two-pass build: 1) build all sheets 2) add cross-refs + save
- Text placed near label in 0.8mm font, offset to avoid overlap

Co-Authored-By: Claude Opus 4.6 <noreply@anthropic.com>
Other:
- note added: "→S01"
- note added: "→S01,S02,S03,S04,S05,S06,S07,S08,S09,S10,S12,S13"
- note added: "→S01,S05"
- note added: "→S01,S06"
- note added: "→S01,S07,S10,S13"
- note added: "→S02,S03"
- note added: "→S02,S03,S04"
- note added: "→S02,S03,S04,S08"
- note added: "→S02,S03,S06"
- note added: "→S02,S03,S06,S13"
- note added: "→S06"
- note added: "→S13"
Changed lines of the file:
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@@
     (effects (font (size 1.000 1.000)))
+  )
+  (text "→S02,S03,S06,S13" (at 65.580 93.940 0)
+    (effects (font (size 0.800 0.800)))
+  )
+  (text "→S02,S03,S06,S13" (at 68.120 180.300 0)
+    (effects (font (size 0.800 0.800)))
+  )
+  (text "→S02,S03,S06" (at 135.080 93.940 0)
+    (effects (font (size 0.800 0.800)))
+  )
+  (text "→S01,S05" (at 135.080 99.020 0)
+    (effects (font (size 0.800 0.800)))
+  )
+  (text "→S01,S02,S03,S04,S05,S06,S07,S08,S09,S10,S12,S13" (at 65.580 85.050 0)
+    (effects (font (size 0.800 0.800)))
+  )
+  (text "→S01,S02,S03,S04,S05,S06,S07,S08,S09,S10,S12,S13" (at 132.540 180.300 0)
+    (effects (font (size 0.800 0.800)))
+  )
+  (text "→S02,S03,S04" (at 264.970 72.350 0)
+    (effects (font (size 0.800 0.800)))
+  )
+  (text "→S02,S03" (at 264.970 77.430 0)
+    (effects (font (size 0.800 0.800)))
+  )
+  (text "→S02,S03" (at 264.970 82.510 0)
+    (effects (font (size 0.800 0.800)))
+  )
+  (text "→S02,S03" (at 264.970 87.590 0)
+    (effects (font (size 0.800 0.800)))
+  )
+  (text "→S02,S03" (at 264.970 92.670 0)
+    (effects (font (size 0.800 0.800)))
+  )
+  (text "→S02,S03" (at 334.470 72.350 0)
+    (effects (font (size 0.800 0.800)))
+  )
+  (text "→S02,S03,S04,S08" (at 334.470 77.430 0)
+    (effects (font (size 0.800 0.800)))
+  )
+  (text "→S02,S03" (at 334.470 82.510 0)
+    (effects (font (size 0.800 0.800)))
+  )
+  (text "→S02,S03" (at 334.470 87.590 0)
+    (effects (font (size 0.800 0.800)))
+  )
+  (text "→S02,S03,S04" (at 334.470 92.670 0)
+    (effects (font (size 0.800 0.800)))
+  )
+  (text "→S01,S07,S10,S13" (at 68.120 185.380 0)
+    (effects (font (size 0.800 0.800)))
+  )
+  (text "→S13" (at 132.540 185.380 0)
+    (effects (font (size 0.800 0.800)))
+  )
+  (text "→S06" (at 270.050 180.300 0)
+    (effects (font (size 0.800 0.800)))
+  )
+  (text "→S01,S06" (at 329.390 180.300 0)
+    (effects (font (size 0.800 0.800)))
+  )
+  (text "→S01" (at 270.050 224.750 0)
+    (effects (font (size 0.800 0.800)))
   )
   (symbol_instances)

Commit message: Fix label text justification for KiCad 9
Add (justify left) to all label and global_label effects.
KiCad 9 requires explicit text justification — without it,
label text is mispositioned relative to the label shape.

Co-Authored-By: Claude Opus 4.6 <noreply@anthropic.com>
Changed lines of the file:
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@@
   )
   (global_label "K_LINE" (shape bidirectional) (at 68.580 91.440 180)
-    (effects (font (size 1.27 1.27)))
+    (effects (font (size 1.27 1.27)) (justify left))
     (property "Intersheetrefs" "${INTERSHEET_REFS}" (at 68.580 91.440 0)
       (effects (font (size 1.27 1.27)) hide)
@@
   )
   (global_label "L_LINE" (shape bidirectional) (at 132.080 91.440 0)
-    (effects (font (size 1.27 1.27)))
+    (effects (font (size 1.27 1.27)) (justify left))
     (property "Intersheetrefs" "${INTERSHEET_REFS}" (at 132.080 91.440 0)
       (effects (font (size 1.27 1.27)) hide)
@@
   )
   (global_label "+12V_ALWAYS" (shape bidirectional) (at 132.080 96.520 0)
-    (effects (font (size 1.27 1.27)))
+    (effects (font (size 1.27 1.27)) (justify left))
     (property "Intersheetrefs" "${INTERSHEET_REFS}" (at 132.080 96.520 0)
       (effects (font (size 1.27 1.27)) hide)
@@
   )
   (global_label "GND" (shape input) (at 68.580 82.550 180)
-    (effects (font (size 1.27 1.27)))
+    (effects (font (size 1.27 1.27)) (justify left))
     (property "Intersheetrefs" "${INTERSHEET_REFS}" (at 68.580 82.550 0)
       (effects (font (size 1.27 1.27)) hide)
@@
   )
   (global_label "DRIVE" (shape bidirectional) (at 267.970 69.850 180)
-    (effects (font (size 1.27 1.27)))
+    (effects (font (size 1.27 1.27)) (justify left))
     (property "Intersheetrefs" "${INTERSHEET_REFS}" (at 267.970 69.850 0)
       (effects (font (size 1.27 1.27)) hide)
@@
   )
   (global_label "START" (shape bidirectional) (at 267.970 74.930 180)
-    (effects (font (size 1.27 1.27)))
+    (effects (font (size 1.27 1.27)) (justify left))
     (property "Intersheetrefs" "${INTERSHEET_REFS}" (at 267.970 74.930 0)
       (effects (font (size 1.27 1.27)) hide)
@@
   )
   (global_label "DRIVE_RDY" (shape bidirectional) (at 267.970 80.010 180)
-    (effects (font (size 1.27 1.27)))
+    (effects (font (size 1.27 1.27)) (justify left))
     (property "Intersheetrefs" "${INTERSHEET_REFS}" (at 267.970 80.010 0)
       (effects (font (size 1.27 1.27)) hide)
@@
   )
   (global_label "FAULT" (shape bidirectional) (at 267.970 85.090 180)
-    (effects (font (size 1.27 1.27)))
+    (effects (font (size 1.27 1.27)) (justify left))
     (property "Intersheetrefs" "${INTERSHEET_REFS}" (at 267.970 85.090 0)
       (effects (font (size 1.27 1.27)) hide)
@@
   )
   (global_label "RED_PWR" (shape bidirectional) (at 267.970 90.170 180)
-    (effects (font (size 1.27 1.27)))
+    (effects (font (size 1.27 1.27)) (justify left))
     (property "Intersheetrefs" "${INTERSHEET_REFS}" (at 267.970 90.170 0)
       (effects (font (size 1.27 1.27)) hide)
@@
   )
   (global_label "BRAKE_SW" (shape bidirectional) (at 331.470 69.850 0)
-    (effects (font (size 1.27 1.27)))
+    (effects (font (size 1.27 1.27)) (justify left))
     (property "Intersheetrefs" "${INTERSHEET_REFS}" (at 331.470 69.850 0)
       (effects (font (size 1.27 1.27)) hide)
@@
   )
   (global_label "REVERSE" (shape bidirectional) (at 331.470 74.930 0)
-    (effects (font (size 1.27 1.27)))
+    (effects (font (size 1.27 1.27)) (justify left))
     (property "Intersheetrefs" "${INTERSHEET_REFS}" (at 331.470 74.930 0)
       (effects (font (size 1.27 1.27)) hide)
@@
   )
   (global_label "GEAR_LOCK" (shape bidirectional) (at 331.470 80.010 0)
-    (effects (font (size 1.27 1.27)))
+    (effects (font (size 1.27 1.27)) (justify left))
     (property "Intersheetrefs" "${INTERSHEET_REFS}" (at 331.470 80.010 0)
       (effects (font (size 1.27 1.27)) hide)
@@
   )
   (global_label "RAD_FAN_CMD" (shape bidirectional) (at 331.470 85.090 0)
-    (effects (font (size 1.27 1.27)))
+    (effects (font (size 1.27 1.27)) (justify left))
     (property "Intersheetrefs" "${INTERSHEET_REFS}" (at 331.470 85.090 0)
       (effects (font (size 1.27 1.27)) hide)
@@
   )
   (global_label "POWER" (shape bidirectional) (at 331.470 90.170 0)
-    (effects (font (size 1.27 1.27)))
+    (effects (font (size 1.27 1.27)) (justify left))
     (property "Intersheetrefs" "${INTERSHEET_REFS}" (at 331.470 90.170 0)
       (effects (font (size 1.27 1.27)) hide)
@@
   )
   (global_label "K_LINE" (shape bidirectional) (at 71.120 177.800 180)
-    (effects (font (size 1.27 1.27)))
+    (effects (font (size 1.27 1.27)) (justify left))
     (property "Intersheetrefs" "${INTERSHEET_REFS}" (at 71.120 177.800 0)
       (effects (font (size 1.27 1.27)) hide)
@@
   )
   (global_label "+12V_F17_COLL_ALM" (shape bidirectional) (at 71.120 182.880 180)
-    (effects (font (size 1.27 1.27)))
+    (effects (font (size 1.27 1.27)) (justify left))
     (property "Intersheetrefs" "${INTERSHEET_REFS}" (at 71.120 182.880 0)
       (effects (font (size 1.27 1.27)) hide)
@@
   )
   (global_label "GND" (shape input) (at 129.540 177.800 0)
-    (effects (font (size 1.27 1.27)))
+    (effects (font (size 1.27 1.27)) (justify left))
     (property "Intersheetrefs" "${INTERSHEET_REFS}" (at 129.540 177.800 0)
       (effects (font (size 1.27 1.27)) hide)
@@
   )
   (global_label "CRASH_SIGNAL" (shape bidirectional) (at 129.540 182.880 0)
-    (effects (font (size 1.27 1.27)))
+    (effects (font (size 1.27 1.27)) (justify left))
     (property "Intersheetrefs" "${INTERSHEET_REFS}" (at 129.540 182.880 0)
       (effects (font (size 1.27 1.27)) hide)
@@
   )
   (global_label "BATT_COOLING" (shape bidirectional) (at 273.050 177.800 180)
-    (effects (font (size 1.27 1.27)))
+    (effects (font (size 1.27 1.27)) (justify left))
     (property "Intersheetrefs" "${INTERSHEET_REFS}" (at 273.050 177.800 0)
       (effects (font (size 1.27 1.27)) hide)
@@
   )
   (global_label "+12V_F10_WPUMP_CHG" (shape bidirectional) (at 326.390 177.800 0)
-    (effects (font (size 1.27 1.27)))
+    (effects (font (size 1.27 1.27)) (justify left))
     (property "Intersheetrefs" "${INTERSHEET_REFS}" (at 326.390 177.800 0)
       (effects (font (size 1.27 1.27)) hide)
@@
   )
   (global_label "SPEED_SIGNAL" (shape bidirectional) (at 273.050 217.170 180)
-    (effects (font (size 1.27 1.27)))
+    (effects (font (size 1.27 1.27)) (justify left))
     (property "Intersheetrefs" "${INTERSHEET_REFS}" (at 273.050 217.170 0)
       (effects (font (size 1.27 1.27)) hide)
@@
   )
   (global_label "+12V_F30_DIAG" (shape bidirectional) (at 273.050 222.250 180)
-    (effects (font (size 1.27 1.27)))
+    (effects (font (size 1.27 1.27)) (justify left))
     (property "Intersheetrefs" "${INTERSHEET_REFS}" (at 273.050 222.250 0)
       (effects (font (size 1.27 1.27)) hide)

Commit message: Relay symbol for flasher, label justify set to auto
- Flasher Relay (Think:FLASHER_RELAY) now has coil+switch graphics
  matching the standard relay symbol style
- All relays (SPST, SPDT, Flasher) use consistent coil+switch body
- Remove (justify left) from all label and global_label effects —
  KiCad 9 auto-determines text alignment based on label orientation

Co-Authored-By: Claude Opus 4.6 <noreply@anthropic.com>
Changed lines of the file:
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@@
   )
   (global_label "K_LINE" (shape bidirectional) (at 68.580 91.440 180)
-    (effects (font (size 1.27 1.27)) (justify left))
+    (effects (font (size 1.27 1.27)))
     (property "Intersheetrefs" "${INTERSHEET_REFS}" (at 68.580 91.440 0)
       (effects (font (size 1.27 1.27)) hide)
@@
   )
   (global_label "L_LINE" (shape bidirectional) (at 132.080 91.440 0)
-    (effects (font (size 1.27 1.27)) (justify left))
+    (effects (font (size 1.27 1.27)))
     (property "Intersheetrefs" "${INTERSHEET_REFS}" (at 132.080 91.440 0)
       (effects (font (size 1.27 1.27)) hide)
@@
   )
   (global_label "+12V_ALWAYS" (shape bidirectional) (at 132.080 96.520 0)
-    (effects (font (size 1.27 1.27)) (justify left))
+    (effects (font (size 1.27 1.27)))
     (property "Intersheetrefs" "${INTERSHEET_REFS}" (at 132.080 96.520 0)
       (effects (font (size 1.27 1.27)) hide)
@@
   )
   (global_label "GND" (shape input) (at 68.580 82.550 180)
-    (effects (font (size 1.27 1.27)) (justify left))
+    (effects (font (size 1.27 1.27)))
     (property "Intersheetrefs" "${INTERSHEET_REFS}" (at 68.580 82.550 0)
       (effects (font (size 1.27 1.27)) hide)
@@
   )
   (global_label "DRIVE" (shape bidirectional) (at 267.970 69.850 180)
-    (effects (font (size 1.27 1.27)) (justify left))
+    (effects (font (size 1.27 1.27)))
     (property "Intersheetrefs" "${INTERSHEET_REFS}" (at 267.970 69.850 0)
       (effects (font (size 1.27 1.27)) hide)
@@
   )
   (global_label "START" (shape bidirectional) (at 267.970 74.930 180)
-    (effects (font (size 1.27 1.27)) (justify left))
+    (effects (font (size 1.27 1.27)))
     (property "Intersheetrefs" "${INTERSHEET_REFS}" (at 267.970 74.930 0)
       (effects (font (size 1.27 1.27)) hide)
@@
   )
   (global_label "DRIVE_RDY" (shape bidirectional) (at 267.970 80.010 180)
-    (effects (font (size 1.27 1.27)) (justify left))
+    (effects (font (size 1.27 1.27)))
     (property "Intersheetrefs" "${INTERSHEET_REFS}" (at 267.970 80.010 0)
       (effects (font (size 1.27 1.27)) hide)
@@
   )
   (global_label "FAULT" (shape bidirectional) (at 267.970 85.090 180)
-    (effects (font (size 1.27 1.27)) (justify left))
+    (effects (font (size 1.27 1.27)))
     (property "Intersheetrefs" "${INTERSHEET_REFS}" (at 267.970 85.090 0)
       (effects (font (size 1.27 1.27)) hide)
@@
   )
   (global_label "RED_PWR" (shape bidirectional) (at 267.970 90.170 180)
-    (effects (font (size 1.27 1.27)) (justify left))
+    (effects (font (size 1.27 1.27)))
     (property "Intersheetrefs" "${INTERSHEET_REFS}" (at 267.970 90.170 0)
       (effects (font (size 1.27 1.27)) hide)
@@
   )
   (global_label "BRAKE_SW" (shape bidirectional) (at 331.470 69.850 0)
-    (effects (font (size 1.27 1.27)) (justify left))
+    (effects (font (size 1.27 1.27)))
     (property "Intersheetrefs" "${INTERSHEET_REFS}" (at 331.470 69.850 0)
       (effects (font (size 1.27 1.27)) hide)
@@
   )
   (global_label "REVERSE" (shape bidirectional) (at 331.470 74.930 0)
-    (effects (font (size 1.27 1.27)) (justify left))
+    (effects (font (size 1.27 1.27)))
     (property "Intersheetrefs" "${INTERSHEET_REFS}" (at 331.470 74.930 0)
       (effects (font (size 1.27 1.27)) hide)
@@
   )
   (global_label "GEAR_LOCK" (shape bidirectional) (at 331.470 80.010 0)
-    (effects (font (size 1.27 1.27)) (justify left))
+    (effects (font (size 1.27 1.27)))
     (property "Intersheetrefs" "${INTERSHEET_REFS}" (at 331.470 80.010 0)
       (effects (font (size 1.27 1.27)) hide)
@@
   )
   (global_label "RAD_FAN_CMD" (shape bidirectional) (at 331.470 85.090 0)
-    (effects (font (size 1.27 1.27)) (justify left))
+    (effects (font (size 1.27 1.27)))
     (property "Intersheetrefs" "${INTERSHEET_REFS}" (at 331.470 85.090 0)
       (effects (font (size 1.27 1.27)) hide)
@@
   )
   (global_label "POWER" (shape bidirectional) (at 331.470 90.170 0)
-    (effects (font (size 1.27 1.27)) (justify left))
+    (effects (font (size 1.27 1.27)))
     (property "Intersheetrefs" "${INTERSHEET_REFS}" (at 331.470 90.170 0)
       (effects (font (size 1.27 1.27)) hide)
@@
   )
   (global_label "K_LINE" (shape bidirectional) (at 71.120 177.800 180)
-    (effects (font (size 1.27 1.27)) (justify left))
+    (effects (font (size 1.27 1.27)))
     (property "Intersheetrefs" "${INTERSHEET_REFS}" (at 71.120 177.800 0)
       (effects (font (size 1.27 1.27)) hide)
@@
   )
   (global_label "+12V_F17_COLL_ALM" (shape bidirectional) (at 71.120 182.880 180)
-    (effects (font (size 1.27 1.27)) (justify left))
+    (effects (font (size 1.27 1.27)))
     (property "Intersheetrefs" "${INTERSHEET_REFS}" (at 71.120 182.880 0)
       (effects (font (size 1.27 1.27)) hide)
@@
   )
   (global_label "GND" (shape input) (at 129.540 177.800 0)
-    (effects (font (size 1.27 1.27)) (justify left))
+    (effects (font (size 1.27 1.27)))
     (property "Intersheetrefs" "${INTERSHEET_REFS}" (at 129.540 177.800 0)
       (effects (font (size 1.27 1.27)) hide)
@@
   )
   (global_label "CRASH_SIGNAL" (shape bidirectional) (at 129.540 182.880 0)
-    (effects (font (size 1.27 1.27)) (justify left))
+    (effects (font (size 1.27 1.27)))
     (property "Intersheetrefs" "${INTERSHEET_REFS}" (at 129.540 182.880 0)
       (effects (font (size 1.27 1.27)) hide)
@@
   )
   (global_label "BATT_COOLING" (shape bidirectional) (at 273.050 177.800 180)
-    (effects (font (size 1.27 1.27)) (justify left))
+    (effects (font (size 1.27 1.27)))
     (property "Intersheetrefs" "${INTERSHEET_REFS}" (at 273.050 177.800 0)
       (effects (font (size 1.27 1.27)) hide)
@@
   )
   (global_label "+12V_F10_WPUMP_CHG" (shape bidirectional) (at 326.390 177.800 0)
-    (effects (font (size 1.27 1.27)) (justify left))
+    (effects (font (size 1.27 1.27)))
     (property "Intersheetrefs" "${INTERSHEET_REFS}" (at 326.390 177.800 0)
       (effects (font (size 1.27 1.27)) hide)
@@
   )
   (global_label "SPEED_SIGNAL" (shape bidirectional) (at 273.050 217.170 180)
-    (effects (font (size 1.27 1.27)) (justify left))
+    (effects (font (size 1.27 1.27)))
     (property "Intersheetrefs" "${INTERSHEET_REFS}" (at 273.050 217.170 0)
       (effects (font (size 1.27 1.27)) hide)
@@
   )
   (global_label "+12V_F30_DIAG" (shape bidirectional) (at 273.050 222.250 180)
-    (effects (font (size 1.27 1.27)) (justify left))
+    (effects (font (size 1.27 1.27)))
     (property "Intersheetrefs" "${INTERSHEET_REFS}" (at 273.050 222.250 0)
       (effects (font (size 1.27 1.27)) hide)
