File: Data/Trabbi Schematic/think_s12_radio_hvac.kicad_sch (KiCad schematic)
At the start: 20 parts, among them K1 Heated RW Relay R2, K2 Blower Relay R12, K3 Recirculation Relay R14, K4 Combustion Heater Relay R16, M1 Brake Vacuum Pump (E14), M2 Heater Blower Motor, M3 Recirculation Motor, SW1 Heater Switch, SW2 Recirculation Switch, SW3 Tailgate Release Switch, U1 Radio Unit, U2 Supplementary Heater (Webasto)

Commit message: Relay symbol for flasher, label justify set to auto
- Flasher Relay (Think:FLASHER_RELAY) now has coil+switch graphics
  matching the standard relay symbol style
- All relays (SPST, SPDT, Flasher) use consistent coil+switch body
- Remove (justify left) from all label and global_label effects —
  KiCad 9 auto-determines text alignment based on label orientation

Co-Authored-By: Claude Opus 4.6 <noreply@anthropic.com>
Changed lines of the file:
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@@
   )
   (global_label "+12V_F7_RADIO" (shape bidirectional) (at 50.800 44.450 180)
-    (effects (font (size 1.27 1.27)) (justify left))
+    (effects (font (size 1.27 1.27)))
     (property "Intersheetrefs" "${INTERSHEET_REFS}" (at 50.800 44.450 0)
       (effects (font (size 1.27 1.27)) hide)
@@
   )
   (global_label "GND" (shape input) (at 50.800 49.530 180)
-    (effects (font (size 1.27 1.27)) (justify left))
+    (effects (font (size 1.27 1.27)))
     (property "Intersheetrefs" "${INTERSHEET_REFS}" (at 50.800 49.530 0)
       (effects (font (size 1.27 1.27)) hide)
@@
   )
   (global_label "GND" (shape input) (at 226.060 35.560 0)
-    (effects (font (size 1.27 1.27)) (justify left))
+    (effects (font (size 1.27 1.27)))
     (property "Intersheetrefs" "${INTERSHEET_REFS}" (at 226.060 35.560 0)
       (effects (font (size 1.27 1.27)) hide)
@@
   )
   (global_label "GND" (shape input) (at 226.060 54.610 0)
-    (effects (font (size 1.27 1.27)) (justify left))
+    (effects (font (size 1.27 1.27)))
     (property "Intersheetrefs" "${INTERSHEET_REFS}" (at 226.060 54.610 0)
       (effects (font (size 1.27 1.27)) hide)
@@
   )
   (label "ANT_SIGNAL" (at 58.420 17.780 0)
-    (effects (font (size 1.27 1.27)) (justify left))
+    (effects (font (size 1.27 1.27)))
   )
   (wire (pts (xy 64.770 54.610) (xy 64.770 20.320))
@@
   )
   (global_label "+12V_F1_HTDWS" (shape bidirectional) (at 113.030 87.630 180)
-    (effects (font (size 1.27 1.27)) (justify left))
+    (effects (font (size 1.27 1.27)))
     (property "Intersheetrefs" "${INTERSHEET_REFS}" (at 113.030 87.630 0)
       (effects (font (size 1.27 1.27)) hide)
@@
   )
   (global_label "GND" (shape input) (at 224.790 90.170 0)
-    (effects (font (size 1.27 1.27)) (justify left))
+    (effects (font (size 1.27 1.27)))
     (property "Intersheetrefs" "${INTERSHEET_REFS}" (at 224.790 90.170 0)
       (effects (font (size 1.27 1.27)) hide)
@@
   )
   (global_label "+12V_F22_VACPUMP" (shape bidirectional) (at 53.340 119.380 180)
-    (effects (font (size 1.27 1.27)) (justify left))
+    (effects (font (size 1.27 1.27)))
     (property "Intersheetrefs" "${INTERSHEET_REFS}" (at 53.340 119.380 0)
       (effects (font (size 1.27 1.27)) hide)
@@
   )
   (global_label "GND" (shape input) (at 106.680 119.380 0)
-    (effects (font (size 1.27 1.27)) (justify left))
+    (effects (font (size 1.27 1.27)))
     (property "Intersheetrefs" "${INTERSHEET_REFS}" (at 106.680 119.380 0)
       (effects (font (size 1.27 1.27)) hide)
@@
   )
   (global_label "+12V_F5_BLOWER" (shape bidirectional) (at 52.070 180.340 180)
-    (effects (font (size 1.27 1.27)) (justify left))
+    (effects (font (size 1.27 1.27)))
     (property "Intersheetrefs" "${INTERSHEET_REFS}" (at 52.070 180.340 0)
       (effects (font (size 1.27 1.27)) hide)
@@
   )
   (global_label "GND" (shape input) (at 248.920 162.560 0)
-    (effects (font (size 1.27 1.27)) (justify left))
+    (effects (font (size 1.27 1.27)))
     (property "Intersheetrefs" "${INTERSHEET_REFS}" (at 248.920 162.560 0)
       (effects (font (size 1.27 1.27)) hide)
@@
   )
   (global_label "+12V_F5_BLOWER" (shape bidirectional) (at 52.070 229.870 180)
-    (effects (font (size 1.27 1.27)) (justify left))
+    (effects (font (size 1.27 1.27)))
     (property "Intersheetrefs" "${INTERSHEET_REFS}" (at 52.070 229.870 0)
       (effects (font (size 1.27 1.27)) hide)
@@
   )
   (global_label "GND" (shape input) (at 273.050 240.030 0)
-    (effects (font (size 1.27 1.27)) (justify left))
+    (effects (font (size 1.27 1.27)))
     (property "Intersheetrefs" "${INTERSHEET_REFS}" (at 273.050 240.030 0)
       (effects (font (size 1.27 1.27)) hide)
@@
   )
   (global_label "+12V_F3_HEATER" (shape bidirectional) (at 321.310 96.520 180)
-    (effects (font (size 1.27 1.27)) (justify left))
+    (effects (font (size 1.27 1.27)))
     (property "Intersheetrefs" "${INTERSHEET_REFS}" (at 321.310 96.520 0)
       (effects (font (size 1.27 1.27)) hide)
@@
   )
   (global_label "GND" (shape input) (at 321.310 104.140 180)
-    (effects (font (size 1.27 1.27)) (justify left))
+    (effects (font (size 1.27 1.27)))
     (property "Intersheetrefs" "${INTERSHEET_REFS}" (at 321.310 104.140 0)
       (effects (font (size 1.27 1.27)) hide)
@@
   )
   (global_label "WEBASTO_CTRL" (shape bidirectional) (at 379.730 105.410 0)
-    (effects (font (size 1.27 1.27)) (justify left))
+    (effects (font (size 1.27 1.27)))
     (property "Intersheetrefs" "${INTERSHEET_REFS}" (at 379.730 105.410 0)
       (effects (font (size 1.27 1.27)) hide)
@@
   )
   (global_label "+12V_F33_WEBASTO" (shape bidirectional) (at 323.850 46.990 180)
-    (effects (font (size 1.27 1.27)) (justify left))
+    (effects (font (size 1.27 1.27)))
     (property "Intersheetrefs" "${INTERSHEET_REFS}" (at 323.850 46.990 0)
       (effects (font (size 1.27 1.27)) hide)
@@
   )
   (global_label "TAILGATE_RELEASE" (shape bidirectional) (at 326.390 170.180 180)
-    (effects (font (size 1.27 1.27)) (justify left))
+    (effects (font (size 1.27 1.27)))
     (property "Intersheetrefs" "${INTERSHEET_REFS}" (at 326.390 170.180 0)
       (effects (font (size 1.27 1.27)) hide)
@@
   )
   (global_label "GND" (shape input) (at 374.650 170.180 0)
-    (effects (font (size 1.27 1.27)) (justify left))
+    (effects (font (size 1.27 1.27)))
     (property "Intersheetrefs" "${INTERSHEET_REFS}" (at 374.650 170.180 0)
       (effects (font (size 1.27 1.27)) hide)
@@
   )
   (global_label "+12V_F9_HORN_DOME" (shape bidirectional) (at 326.390 199.390 180)
-    (effects (font (size 1.27 1.27)) (justify left))
+    (effects (font (size 1.27 1.27)))
     (property "Intersheetrefs" "${INTERSHEET_REFS}" (at 326.390 199.390 0)
       (effects (font (size 1.27 1.27)) hide)
