File: Data/Trabbi Schematic/think_s13_safety_hv.kicad_sch (KiCad schematic)
At the start: 5 parts, among them U1 Collision Control Unit (C050), U2 Contactor Box Internal Detail, U3 HV Distribution Box Detail

Commit message: Relay symbol for flasher, label justify set to auto
- Flasher Relay (Think:FLASHER_RELAY) now has coil+switch graphics
  matching the standard relay symbol style
- All relays (SPST, SPDT, Flasher) use consistent coil+switch body
- Remove (justify left) from all label and global_label effects —
  KiCad 9 auto-determines text alignment based on label orientation

Co-Authored-By: Claude Opus 4.6 <noreply@anthropic.com>
Changed lines of the file:
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@@
   )
   (global_label "K_LINE" (shape bidirectional) (at 68.580 52.070 180)
-    (effects (font (size 1.27 1.27)) (justify left))
+    (effects (font (size 1.27 1.27)))
     (property "Intersheetrefs" "${INTERSHEET_REFS}" (at 68.580 52.070 0)
       (effects (font (size 1.27 1.27)) hide)
@@
   )
   (global_label "+12V_F17_COLL_ALM" (shape output) (at 68.580 59.690 180)
-    (effects (font (size 1.27 1.27)) (justify left))
+    (effects (font (size 1.27 1.27)))
     (property "Intersheetrefs" "${INTERSHEET_REFS}" (at 68.580 59.690 0)
       (effects (font (size 1.27 1.27)) hide)
@@
   )
   (global_label "CRASH_SIGNAL" (shape bidirectional) (at 68.580 67.310 180)
-    (effects (font (size 1.27 1.27)) (justify left))
+    (effects (font (size 1.27 1.27)))
     (property "Intersheetrefs" "${INTERSHEET_REFS}" (at 68.580 67.310 0)
       (effects (font (size 1.27 1.27)) hide)
@@
   )
   (global_label "WARNING_LAMP" (shape bidirectional) (at 132.080 62.230 0)
-    (effects (font (size 1.27 1.27)) (justify left))
+    (effects (font (size 1.27 1.27)))
     (property "Intersheetrefs" "${INTERSHEET_REFS}" (at 132.080 62.230 0)
       (effects (font (size 1.27 1.27)) hide)
@@
   )
   (global_label "GND" (shape input) (at 132.080 68.580 0)
-    (effects (font (size 1.27 1.27)) (justify left))
+    (effects (font (size 1.27 1.27)))
     (property "Intersheetrefs" "${INTERSHEET_REFS}" (at 132.080 68.580 0)
       (effects (font (size 1.27 1.27)) hide)
@@
   )
   (global_label "GND" (shape input) (at 276.860 44.450 0)
-    (effects (font (size 1.27 1.27)) (justify left))
+    (effects (font (size 1.27 1.27)))
     (property "Intersheetrefs" "${INTERSHEET_REFS}" (at 276.860 44.450 0)
       (effects (font (size 1.27 1.27)) hide)
@@
   )
   (global_label "GND" (shape input) (at 276.860 64.770 0)
-    (effects (font (size 1.27 1.27)) (justify left))
+    (effects (font (size 1.27 1.27)))
     (property "Intersheetrefs" "${INTERSHEET_REFS}" (at 276.860 64.770 0)
       (effects (font (size 1.27 1.27)) hide)
@@
   )
   (global_label "+114V" (shape bidirectional) (at 152.400 153.670 180)
-    (effects (font (size 1.27 1.27)) (justify left))
+    (effects (font (size 1.27 1.27)))
     (property "Intersheetrefs" "${INTERSHEET_REFS}" (at 152.400 153.670 0)
       (effects (font (size 1.27 1.27)) hide)
@@
   )
   (global_label "-114V" (shape bidirectional) (at 152.400 167.640 180)
-    (effects (font (size 1.27 1.27)) (justify left))
+    (effects (font (size 1.27 1.27)))
     (property "Intersheetrefs" "${INTERSHEET_REFS}" (at 152.400 167.640 0)
       (effects (font (size 1.27 1.27)) hide)
@@
   )
   (label "MAIN_RELAY_COIL" (at 152.400 180.340 0)
-    (effects (font (size 1.27 1.27)) (justify left))
+    (effects (font (size 1.27 1.27)))
   )
   (wire (pts (xy 165.100 193.040) (xy 152.400 193.040))
@@
   )
   (label "AUX_RELAY_COIL" (at 152.400 193.040 0)
-    (effects (font (size 1.27 1.27)) (justify left))
+    (effects (font (size 1.27 1.27)))
   )
   (wire (pts (xy 165.100 207.010) (xy 152.400 207.010))
@@
   )
   (label "HEATER_RELAY_COIL" (at 152.400 207.010 0)
-    (effects (font (size 1.27 1.27)) (justify left))
+    (effects (font (size 1.27 1.27)))
   )
   (wire (pts (xy 233.680 153.670) (xy 246.380 153.670))
@@
   )
   (global_label "+114V_TO_MC" (shape bidirectional) (at 246.380 153.670 0)
-    (effects (font (size 1.27 1.27)) (justify left))
+    (effects (font (size 1.27 1.27)))
     (property "Intersheetrefs" "${INTERSHEET_REFS}" (at 246.380 153.670 0)
       (effects (font (size 1.27 1.27)) hide)
@@
   )
   (global_label "-114V_TO_MC" (shape bidirectional) (at 246.380 167.640 0)
-    (effects (font (size 1.27 1.27)) (justify left))
+    (effects (font (size 1.27 1.27)))
     (property "Intersheetrefs" "${INTERSHEET_REFS}" (at 246.380 167.640 0)
       (effects (font (size 1.27 1.27)) hide)
@@
   )
   (label "PRECHARGE_OUT" (at 246.380 180.340 0)
-    (effects (font (size 1.27 1.27)) (justify left))
+    (effects (font (size 1.27 1.27)))
   )
   (wire (pts (xy 233.680 193.040) (xy 246.380 193.040))
@@
   )
   (global_label "LEM_SENSE+" (shape bidirectional) (at 246.380 193.040 0)
-    (effects (font (size 1.27 1.27)) (justify left))
+    (effects (font (size 1.27 1.27)))
     (property "Intersheetrefs" "${INTERSHEET_REFS}" (at 246.380 193.040 0)
       (effects (font (size 1.27 1.27)) hide)
@@
   )
   (global_label "LEM_SENSE-" (shape bidirectional) (at 246.380 207.010 0)
-    (effects (font (size 1.27 1.27)) (justify left))
+    (effects (font (size 1.27 1.27)))
     (property "Intersheetrefs" "${INTERSHEET_REFS}" (at 246.380 207.010 0)
       (effects (font (size 1.27 1.27)) hide)
@@
   )
   (global_label "CB_RUN" (shape bidirectional) (at 220.980 124.460 90)
-    (effects (font (size 1.27 1.27)) (justify left))
+    (effects (font (size 1.27 1.27)))
     (property "Intersheetrefs" "${INTERSHEET_REFS}" (at 220.980 124.460 0)
       (effects (font (size 1.27 1.27)) hide)
@@
   )
   (global_label "BMS_CMD" (shape bidirectional) (at 212.090 124.460 90)
-    (effects (font (size 1.27 1.27)) (justify left))
+    (effects (font (size 1.27 1.27)))
     (property "Intersheetrefs" "${INTERSHEET_REFS}" (at 212.090 124.460 0)
       (effects (font (size 1.27 1.27)) hide)
@@
   )
   (global_label "CHG_START" (shape bidirectional) (at 203.200 124.460 90)
-    (effects (font (size 1.27 1.27)) (justify left))
+    (effects (font (size 1.27 1.27)))
     (property "Intersheetrefs" "${INTERSHEET_REFS}" (at 203.200 124.460 0)
       (effects (font (size 1.27 1.27)) hide)
@@
   )
   (global_label "PREHEAT" (shape bidirectional) (at 195.580 124.460 90)
-    (effects (font (size 1.27 1.27)) (justify left))
+    (effects (font (size 1.27 1.27)))
     (property "Intersheetrefs" "${INTERSHEET_REFS}" (at 195.580 124.460 0)
       (effects (font (size 1.27 1.27)) hide)
@@
   )
   (global_label "CHARGE" (shape bidirectional) (at 186.690 124.460 90)
-    (effects (font (size 1.27 1.27)) (justify left))
+    (effects (font (size 1.27 1.27)))
     (property "Intersheetrefs" "${INTERSHEET_REFS}" (at 186.690 124.460 0)
       (effects (font (size 1.27 1.27)) hide)
@@
   )
   (global_label "+12V_F28_DRIVE" (shape bidirectional) (at 177.800 124.460 90)
-    (effects (font (size 1.27 1.27)) (justify left))
+    (effects (font (size 1.27 1.27)))
     (property "Intersheetrefs" "${INTERSHEET_REFS}" (at 177.800 124.460 0)
       (effects (font (size 1.27 1.27)) hide)
@@
   )
   (global_label "GND" (shape input) (at 209.550 233.680 270)
-    (effects (font (size 1.27 1.27)) (justify left))
+    (effects (font (size 1.27 1.27)))
     (property "Intersheetrefs" "${INTERSHEET_REFS}" (at 209.550 233.680 0)
       (effects (font (size 1.27 1.27)) hide)
@@
   )
   (global_label "DIAG_CB" (shape bidirectional) (at 189.230 233.680 270)
-    (effects (font (size 1.27 1.27)) (justify left))
+    (effects (font (size 1.27 1.27)))
     (property "Intersheetrefs" "${INTERSHEET_REFS}" (at 189.230 233.680 0)
       (effects (font (size 1.27 1.27)) hide)
@@
   )
   (global_label "+114V" (shape bidirectional) (at 22.860 193.040 180)
-    (effects (font (size 1.27 1.27)) (justify left))
+    (effects (font (size 1.27 1.27)))
     (property "Intersheetrefs" "${INTERSHEET_REFS}" (at 22.860 193.040 0)
       (effects (font (size 1.27 1.27)) hide)
@@
   )
   (global_label "-114V" (shape bidirectional) (at 22.860 205.740 180)
-    (effects (font (size 1.27 1.27)) (justify left))
+    (effects (font (size 1.27 1.27)))
     (property "Intersheetrefs" "${INTERSHEET_REFS}" (at 22.860 205.740 0)
       (effects (font (size 1.27 1.27)) hide)
@@
   )
   (label "VA_CB+" (at 96.520 185.420 0)
-    (effects (font (size 1.27 1.27)) (justify left))
+    (effects (font (size 1.27 1.27)))
   )
   (wire (pts (xy 83.820 190.500) (xy 96.520 190.500))
@@
   )
   (label "VB_CB-" (at 96.520 190.500 0)
-    (effects (font (size 1.27 1.27)) (justify left))
+    (effects (font (size 1.27 1.27)))
   )
   (wire (pts (xy 83.820 196.850) (xy 96.520 196.850))
@@
   )
   (label "VD_DCDC+" (at 96.520 196.850 0)
-    (effects (font (size 1.27 1.27)) (justify left))
+    (effects (font (size 1.27 1.27)))
   )
   (wire (pts (xy 83.820 201.930) (xy 96.520 201.930))
@@
   )
   (label "VD_DCDC-" (at 96.520 201.930 0)
-    (effects (font (size 1.27 1.27)) (justify left))
+    (effects (font (size 1.27 1.27)))
   )
   (wire (pts (xy 83.820 208.280) (xy 96.520 208.280))
@@
   )
   (label "VQ_CHG+" (at 96.520 208.280 0)
-    (effects (font (size 1.27 1.27)) (justify left))
+    (effects (font (size 1.27 1.27)))
   )
   (wire (pts (xy 83.820 213.360) (xy 96.520 213.360))
@@
   )
   (label "VQ_CHG-" (at 96.520 213.360 0)
-    (effects (font (size 1.27 1.27)) (justify left))
+    (effects (font (size 1.27 1.27)))
   )
   (wire (pts (xy 66.040 175.260) (xy 66.040 165.100))
@@
   )
   (label "VH_HEAT" (at 66.040 165.100 0)
-    (effects (font (size 1.27 1.27)) (justify left))
+    (effects (font (size 1.27 1.27)))
   )
   (wire (pts (xy 53.340 175.260) (xy 53.340 165.100))
@@
   )
   (label "VK_CTRL" (at 53.340 165.100 0)
-    (effects (font (size 1.27 1.27)) (justify left))
+    (effects (font (size 1.27 1.27)))
   )
   (text "SAFETY SYSTEMS & HV DETAIL" (at 30.000 260.000 0)
